Commit message: Update me6_robot.urdf

File: dobot_rviz/urdf/me6_robot.urdf (robot description, URDF)
Before this commit: robot me6_robot, 8 links, 7 joints
Links:
- link Link1: geometry collision mesh filename=package://dobot_rviz/meshes/me6/Link1.STL; visual mesh filename=package://dobot_rviz/meshes/me6/Link1.STL
- link Link2: geometry collision mesh filename=package://dobot_rviz/meshes/me6/Link2.STL; visual mesh filename=package://dobot_rviz/meshes/me6/Link2.STL
- link Link3: geometry collision mesh filename=package://dobot_rviz/meshes/me6/Link3.STL; visual mesh filename=package://dobot_rviz/meshes/me6/Link3.STL
- link Link4: geometry collision mesh filename=package://dobot_rviz/meshes/me6/Link4.STL; visual mesh filename=package://dobot_rviz/meshes/me6/Link4.STL
- link Link5: geometry collision mesh filename=package://dobot_rviz/meshes/me6/Link5.STL; visual mesh filename=package://dobot_rviz/meshes/me6/Link5.STL
- link Link6: geometry collision mesh filename=package://dobot_rviz/meshes/me6/Link6.STL; visual mesh filename=package://dobot_rviz/meshes/me6/Link6.STL
- link base_link: geometry collision mesh filename=package://dobot_rviz/meshes/me6/base_link.STL; visual mesh filename=package://dobot_rviz/meshes/me6/base_link.STL
