Commit message: Version_Update

File: cra_description/urdf/cr10_robot.xacro (robot description, xacro)
@@ -104,6 +104,6 @@
       xyz="0 0 1" />
     <limit
-      lower="-3.14"
-      upper="3.14"
+      lower="-6.27"
+      upper="6.27"
       effort="300"
       velocity="100" />
@@ -162,6 +162,6 @@
       xyz="0 0 1" />
     <limit
-      lower="-3.14"
-      upper="3.14"
+      lower="-6.27"
+      upper="6.27"
       effort="300"
       velocity="100" />
@@ -278,6 +278,6 @@
       xyz="0 0 1" />
     <limit
-      lower="-3.14"
-      upper="3.14"
+      lower="-6.27"
+      upper="6.27"
       effort="300"
       velocity="100" />
@@ -336,6 +336,6 @@
       xyz="0 0 1" />
     <limit
-      lower="-3.14"
-      upper="3.14"
+      lower="-6.27"
+      upper="6.27"
       effort="300"
       velocity="100" />
@@ -394,6 +394,6 @@
       xyz="0 0 1" />
     <limit
-      lower="-6.28"
-      upper="6.28"
+      lower="-6.27"
+      upper="6.27"
       effort="300"
       velocity="100" />

File: cra_description/urdf/cr12_robot.xacro (robot description, xacro)
@@ -108,6 +108,6 @@
       xyz="0 0 1" />
     <limit
-      lower="-6.28"
-      upper="6.28"
+      lower="-6.27"
+      upper="6.27"
       effort="300"
       velocity="100" />
@@ -166,6 +166,6 @@
       xyz="0 0 1" />
     <limit
-      lower="-6.28"
-      upper="6.28"
+      lower="-6.27"
+      upper="6.27"
       effort="300"
       velocity="100" />
@@ -282,6 +282,6 @@
       xyz="0 0 1" />
     <limit
-      lower="-6.28"
-      upper="6.28"
+      lower="-6.27"
+      upper="6.27"
       effort="300"
       velocity="100" />
@@ -340,6 +340,6 @@
       xyz="0 0 0.999999999998195" />
     <limit
-      lower="-6.28"
-      upper="6.28"
+      lower="-6.27"
+      upper="6.27"
       effort="300"
       velocity="100" />
@@ -398,6 +398,6 @@
       xyz="0 0 1" />
     <limit
-      lower="-6.28"
-      upper="6.28"
+      lower="-6.27"
+      upper="6.27"
       effort="300"
       velocity="100" />

File: cra_description/urdf/cr16_robot.xacro (robot description, xacro)
@@ -104,6 +104,6 @@
       xyz="0 0 1" />
     <limit
-      lower="-3.14"
-      upper="3.14"
+      lower="-6.27"
+      upper="6.27"
       effort="300"
       velocity="100" />
@@ -162,6 +162,6 @@
       xyz="0 0 1" />
     <limit
-      lower="-3.14"
-      upper="3.14"
+      lower="-6.27"
+      upper="6.27"
       effort="300"
       velocity="100" />
@@ -278,6 +278,6 @@
       xyz="0 0 1" />
     <limit
-      lower="-3.14"
-      upper="3.14"
+      lower="-6.27"
+      upper="6.27"
       effort="300"
       velocity="100" />
@@ -336,6 +336,6 @@
       xyz="0 0 1" />
     <limit
-      lower="-3.14"
-      upper="3.14"
+      lower="-6.27"
+      upper="6.27"
       effort="300"
       velocity="100" />
@@ -394,6 +394,6 @@
       xyz="0 0 1" />
     <limit
-      lower="-6.28"
-      upper="6.28"
+      lower="-6.27"
+      upper="6.27"
       effort="300"
       velocity="100" />

File: cra_description/urdf/cr3_robot.xacro (robot description, xacro)
@@ -104,6 +104,6 @@
       xyz="0 0 1" />
     <limit
-      lower="-3.14"
-      upper="3.14"
+      lower="-6.27"
+      upper="6.27"
       effort="300"
       velocity="100" />
@@ -162,6 +162,6 @@
       xyz="0 0 1" />
     <limit
-      lower="-3.14"
-      upper="3.14"
+      lower="-6.27"
+      upper="6.27"
       effort="300"
       velocity="100" />
@@ -278,6 +278,6 @@
       xyz="0 0 1" />
     <limit
-      lower="-3.14"
-      upper="3.14"
+      lower="-6.27"
+      upper="6.27"
       effort="300"
       velocity="100" />
@@ -336,6 +336,6 @@
       xyz="0 0 1" />
     <limit
-      lower="-3.14"
-      upper="3.14"
+      lower="-6.27"
+      upper="6.27"
       effort="300"
       velocity="100" />
@@ -394,6 +394,6 @@
       xyz="0 0 1" />
     <limit
-      lower="-6.28"
-      upper="6.28"
+      lower="-6.27"
+      upper="6.27"
       effort="300"
       velocity="100" />

File: cra_description/urdf/cr5_robot.xacro (robot description, xacro)
@@ -74,5 +74,5 @@
     <child link="Link1" />
     <axis xyz="0 0 1" />
-    <limit lower="-3.14" upper="3.14" effort="300" velocity="100" />
+    <limit lower="-6.27" upper="6.27" effort="300" velocity="100" />
   </joint>
   <link name="Link2">
@@ -110,5 +110,5 @@
     <child  link="Link2" />
     <axis xyz="0 0 1" />
-    <limit lower="-3.14" upper="3.14" effort="300" velocity="100" />
+    <limit lower="-6.27" upper="6.27" effort="300" velocity="100" />
   </joint>
   <link name="Link3">
@@ -181,5 +181,5 @@
     <child link="Link4" />
     <axis xyz="0 0 1" />
-    <limit lower="-3.14" upper="3.14" effort="300" velocity="100" />
+    <limit lower="-6.27" upper="6.27" effort="300" velocity="100" />
   </joint>
   <link
@@ -217,5 +217,5 @@
     <child link="Link5" />
     <axis xyz="0 0 1" />
-    <limit lower="-3.14" upper="3.14" effort="300" velocity="100" />
+    <limit lower="-6.27" upper="6.27" effort="300" velocity="100" />
   </joint>
   <link name="Link6">
@@ -252,5 +252,5 @@
     <child link="Link6" />
     <axis xyz="0 0 1" />
-    <limit lower="-6.28" upper="6.28" effort="300" velocity="100" />
+    <limit lower="-6.27" upper="6.27" effort="300" velocity="100" />
   </joint>
     <gazebo reference="base_link">

File: cra_description/urdf/cr7_robot.xacro (robot description, xacro)
@@ -107,6 +107,6 @@
       xyz="0 0 -1" />
     <limit
-      lower="-6.28"
-      upper="6.28"
+      lower="-6.27"
+      upper="6.27"
       effort="300"
       velocity="100" />
@@ -165,6 +165,6 @@
       xyz="0 0 1" />
     <limit
-      lower="-6.28"
-      upper="6.28"
+      lower="-6.27"
+      upper="6.27"
       effort="300"
       velocity="100" />
@@ -281,6 +281,6 @@
       xyz="0 0 0.999999999969965" />
     <limit
-      lower="-6.28"
-      upper="6.28"
+      lower="-6.27"
+      upper="6.27"
       effort="300"
       velocity="100" />
@@ -339,6 +339,6 @@
       xyz="0 0 -1" />
     <limit
-      lower="-6.28"
-      upper="6.28"
+      lower="-6.27"
+      upper="6.27"
       effort="300"
       velocity="100" />
@@ -397,6 +397,6 @@
       xyz="0 0 -1" />
     <limit
-      lower="-6.28"
-      upper="6.28"
+      lower="-6.27"
+      upper="6.27"
       effort="300"
       velocity="100" />

File: cra_description/urdf/me6_robot.xacro (robot description, xacro)
@@ -55,5 +55,5 @@
         <child link="Link1" />
         <axis xyz="0 0 1" />
-        <limit lower="-6.28" upper="6.28" effort="300" velocity="300" />
+        <limit lower="-6.27" upper="6.27" effort="300" velocity="300" />
     </joint>
     <link name="Link2">
@@ -200,5 +200,5 @@
         <child link="Link6" />
         <axis xyz="0 0 1" />
-        <limit lower="-6.28" upper="6.28" effort="300" velocity="300" />
+        <limit lower="-6.27" upper="6.27" effort="300" velocity="300" />
     </joint>
    <link name="world" />

File: cra_description/urdf/nova2_robot.xacro (robot description, xacro)
@@ -302,5 +302,5 @@
     <gazebo>
         <plugin filename="libgazebo_ros2_control.so" name="gazebo_ros2_control">
-            <parameters>/home/dobot/V4_ROS2_ws/src/DOBOT_6Axis_ROS2/cr5_moveit/config/ros2_controllers.yaml</parameters>
+            <parameters> $(find nova2_moveit)/config/ros2_controllers.yaml</parameters>
             <robot_param_node>robot_state_publisher</robot_param_node>
         </plugin>

File: cra_description/urdf/nova5_robot.xacro (robot description, xacro)
@@ -495,5 +495,5 @@
     <gazebo>
         <plugin filename="libgazebo_ros2_control.so" name="gazebo_ros2_control">
-            <parameters>/home/dobot/V4_ROS2_ws/src/DOBOT_6Axis_ROS2/cr5_moveit/config/ros2_controllers.yaml</parameters>
+            <parameters> $(find nova5_moveit)/config/ros2_controllers.yaml</parameters>
             <robot_param_node>robot_state_publisher</robot_param_node>
         </plugin>

File: dobot_rviz/urdf/cr10_robot.urdf (robot description, URDF)
Before this commit: robot cr10_robot, 8 links, 7 joints
Joints:
- joint joint1: limit lower=-3.14 upper=3.14 effort=0 velocity=0 -> lower=-6.27 upper=6.27 effort=0 velocity=0
- joint joint2: limit lower=-3.14 upper=3.14 effort=0 velocity=0 -> lower=-6.27 upper=6.27 effort=0 velocity=0
- joint joint4: limit lower=-3.14 upper=3.14 effort=0 velocity=0 -> lower=-6.27 upper=6.27 effort=0 velocity=0
- joint joint5: limit lower=-3.14 upper=3.14 effort=0 velocity=0 -> lower=-6.27 upper=6.27 effort=0 velocity=0
- joint joint6: limit lower=-6.28 upper=6.28 effort=0 velocity=0 -> lower=-6.27 upper=6.27 effort=0 velocity=0

File: dobot_rviz/urdf/cr12_robot.urdf (robot description, URDF)
Before this commit: robot cr12_robot, 8 links, 7 joints
Joints:
- joint joint1: limit lower=-6.28 upper=6.28 effort=0 velocity=0 -> lower=-6.27 upper=6.27 effort=0 velocity=0
- joint joint2: limit lower=-6.28 upper=6.28 effort=0 velocity=0 -> lower=-6.27 upper=6.27 effort=0 velocity=0
- joint joint4: limit lower=-6.28 upper=6.28 effort=0 velocity=0 -> lower=-6.27 upper=6.27 effort=0 velocity=0
- joint joint5: limit lower=-6.28 upper=6.28 effort=0 velocity=0 -> lower=-6.27 upper=6.27 effort=0 velocity=0
- joint joint6: limit lower=-6.28 upper=6.28 effort=0 velocity=0 -> lower=-6.27 upper=6.27 effort=0 velocity=0

File: dobot_rviz/urdf/cr16_robot.urdf (robot description, URDF)
Before this commit: robot cr16_robot, 8 links, 7 joints
Joints:
- joint joint1: limit lower=-3.14 upper=3.14 effort=0 velocity=0 -> lower=-6.27 upper=6.27 effort=0 velocity=0
- joint joint2: limit lower=-3.14 upper=3.14 effort=0 velocity=0 -> lower=-6.27 upper=6.27 effort=0 velocity=0
- joint joint4: limit lower=-3.14 upper=3.14 effort=0 velocity=0 -> lower=-6.27 upper=6.27 effort=0 velocity=0
- joint joint5: limit lower=-3.14 upper=3.14 effort=0 velocity=0 -> lower=-6.27 upper=6.27 effort=0 velocity=0
- joint joint6: limit lower=-6.28 upper=6.28 effort=0 velocity=0 -> lower=-6.27 upper=6.27 effort=0 velocity=0

File: dobot_rviz/urdf/cr3_robot.urdf (robot description, URDF)
Before this commit: robot cr3_robot, 8 links, 7 joints
Joints:
- joint joint1: limit lower=-3.14 upper=3.14 effort=0 velocity=0 -> lower=-6.27 upper=6.27 effort=0 velocity=0
- joint joint2: limit lower=-3.14 upper=3.14 effort=0 velocity=0 -> lower=-6.27 upper=6.27 effort=0 velocity=0
- joint joint4: limit lower=-3.14 upper=3.14 effort=0 velocity=0 -> lower=-6.27 upper=6.27 effort=0 velocity=0
- joint joint5: limit lower=-3.14 upper=3.14 effort=0 velocity=0 -> lower=-6.27 upper=6.27 effort=0 velocity=0
- joint joint6: limit lower=-6.28 upper=6.28 effort=0 velocity=0 -> lower=-6.27 upper=6.27 effort=0 velocity=0

File: dobot_rviz/urdf/cr5_robot.urdf (robot description, URDF)
Before this commit: robot cr5_robot, 8 links, 7 joints
Joints:
- joint joint1: limit lower=-3.14 upper=3.14 effort=0 velocity=0 -> lower=-6.27 upper=6.27 effort=0 velocity=0
- joint joint2: limit lower=-3.14 upper=3.14 effort=0 velocity=0 -> lower=-6.27 upper=6.27 effort=0 velocity=0
- joint joint4: limit lower=-3.14 upper=3.14 effort=0 velocity=0 -> lower=-6.27 upper=6.27 effort=0 velocity=0
- joint joint5: limit lower=-3.14 upper=3.14 effort=0 velocity=0 -> lower=-6.27 upper=6.27 effort=0 velocity=0
- joint joint6: limit lower=-6.28 upper=6.28 effort=0 velocity=0 -> lower=-6.27 upper=6.27 effort=0 velocity=0

File: dobot_rviz/urdf/cr7_robot.urdf (robot description, URDF)
Before this commit: robot cr7_robot, 8 links, 7 joints
Joints:
- joint joint1: limit lower=-6.28 upper=6.28 effort=0 velocity=0 -> lower=-6.27 upper=6.27 effort=0 velocity=0
- joint joint2: limit lower=-6.28 upper=6.28 effort=0 velocity=0 -> lower=-6.27 upper=6.27 effort=0 velocity=0
- joint joint4: limit lower=-6.28 upper=6.28 effort=0 velocity=0 -> lower=-6.27 upper=6.27 effort=0 velocity=0
- joint joint5: limit lower=-6.28 upper=6.28 effort=0 velocity=0 -> lower=-6.27 upper=6.27 effort=0 velocity=0
- joint joint6: limit lower=-6.28 upper=6.28 effort=0 velocity=0 -> lower=-6.27 upper=6.27 effort=0 velocity=0

File: dobot_rviz/urdf/me6_robot.urdf (robot description, URDF)
Before this commit: robot me6_robot, 8 links, 7 joints
Joints:
- joint joint1: limit lower=-6.28 upper=6.28 effort=0 velocity=0 -> lower=-6.27 upper=6.27 effort=0 velocity=0
- joint joint6: limit lower=-6.28 upper=6.28 effort=0 velocity=0 -> lower=-6.27 upper=6.27 effort=0 velocity=0
