Commit message: Add CR30H

File: cra_description/urdf/cr10_robot.xacro (robot description, xacro)
@@ -44,4 +44,5 @@
   <link  name="world"/>
 <joint name="world_joint" type="fixed">
+    <origin xyz="0 0 0.03" rpy="0 0 0" />
     <parent link="world" />
     <child  link="dummy_link" />

File: cra_description/urdf/cr12_robot.xacro (robot description, xacro)
@@ -48,4 +48,5 @@
   <link  name="world"/>
 <joint name="world_joint" type="fixed">
+    <origin xyz="0 0 0.03" rpy="0 0 0" />
     <parent link="world" />
     <child  link="dummy_link" />

File: cra_description/urdf/cr16_robot.xacro (robot description, xacro)
@@ -44,4 +44,5 @@
   <link  name="world"/>
 <joint name="world_joint" type="fixed">
+    <origin xyz="0 0 0.03" rpy="0 0 0" />
     <parent link="world" />
     <child  link="dummy_link" />

File: cra_description/urdf/cr30h_robot.xacro (robot description, xacro)
@@ -1,5 +1,5 @@
 <?xml version="1.0" encoding="utf-8"?>
 <robot
-  name="cr20_robot" xmlns:xacro="http://ros.org/wiki/xacro">
+  name="cr30h_robot" xmlns:xacro="http://ros.org/wiki/xacro">
   <link name="dummy_link"/>
   <link
@@ -7,41 +7,41 @@
     <inertial>
       <origin
-        xyz="-0.0523349568972135 0.0899270486094572 -0.00279275668479641"
-        rpy="0 0 0" />
-      <mass
-        value="0.00264393848129463" />
-      <inertia
-        ixx="0"
-        ixy="0"
-        ixz="0"
-        iyy="0"
-        iyz="0"
-        izz="0" />
-    </inertial>
-    <visual>
-      <origin
-        xyz="0 0 0"
-        rpy="0 0 0" />
-      <geometry>
-        <mesh
-          filename="file://$(find cra_description)/meshes/cr20/base_link.STL" />
-      </geometry>
-      <material
-        name="">
-        <color
-          rgba="0.792156862745098 0.819607843137255 0.933333333333333 1" />
-      </material>
-    </visual>
-    <collision>
-      <origin
-        xyz="0 0 0"
-        rpy="0 0 0" />
-      <geometry>
-        <mesh
-          filename="file://$(find cra_description)/meshes/cr20/base_link.STL" />
-      </geometry>
-    </collision>
-  </link>
-    <link  name="world"/>
+        xyz="-1.78212555854348E-05 0.00033084177723393 0.0931967971971018"
+        rpy="0 0 0" />
+      <mass
+        value="3.62558882362798" />
+      <inertia
+        ixx="0.0188475732650718"
+        ixy="-1.37313910460006E-06"
+        ixz="-4.46309791436276E-06"
+        iyy="0.0186121426737853"
+        iyz="7.17633946778761E-05"
+        izz="0.0272514849943692" />
+    </inertial>
+    <visual>
+      <origin
+        xyz="0 0 0"
+        rpy="0 0 0" />
+      <geometry>
+        <mesh
+          filename="file://$(find cra_description)/meshes/cr30h/base_link.STL" />
+      </geometry>
+      <material
+        name="">
+        <color
+          rgba="1 1 1 1" />
+      </material>
+    </visual>
+    <collision>
+      <origin
+        xyz="0 0 0"
+        rpy="0 0 0" />
+      <geometry>
+        <mesh
+          filename="file://$(find cra_description)/meshes/cr30h/base_link.STL" />
+      </geometry>
+    </collision>
+  </link>
+  <link  name="world"/>
   <joint name="world_joint" type="fixed">
     <origin xyz="0 0 0.03" rpy="0 0 0" />
@@ -50,44 +50,44 @@
   </joint>
   <joint name="dummy_joint" type="fixed">
-    <parent link="dummy_link" />
-    <child  link="base_link" />
-  </joint>
+      <parent link="dummy_link" />
+      <child  link="base_link" />
+    </joint>
   <link
     name="Link1">
     <inertial>
       <origin
-        xyz="-0.0154576425326206 -0.0986375365415087 1.04119647925812"
-        rpy="0 0 0" />
-      <mass
-        value="0.00895254328755396" />
-      <inertia
-        ixx="0"
-        ixy="0"
-        ixz="0"
-        iyy="0"
-        iyz="0"
-        izz="0" />
-    </inertial>
-    <visual>
-      <origin
-        xyz="0 0 0"
-        rpy="0 0 0" />
-      <geometry>
-        <mesh
-          filename="file://$(find cra_description)/meshes/cr20/Link1.STL" />
-      </geometry>
-      <material
-        name="">
-        <color
-          rgba="0.792156862745098 0.819607843137255 0.933333333333333 1" />
-      </material>
-    </visual>
-    <collision>
-      <origin
-        xyz="0 0 0"
-        rpy="0 0 0" />
-      <geometry>
-        <mesh
-          filename="file://$(find cra_description)/meshes/cr20/Link1.STL" />
+        xyz="0.0685683156633234 6.45617962612603E-06 0.0352475118413176"
+        rpy="0 0 0" />
+      <mass
+        value="14.4147388577882" />
+      <inertia
+        ixx="0.117399762147082"
+        ixy="-1.3100541842346E-07"
+        ixz="0.0356431430537303"
+        iyy="0.187002726933162"
+        iyz="6.38547998155339E-07"
+        izz="0.161038602803283" />
+    </inertial>
+    <visual>
+      <origin
+        xyz="0 0 0"
+        rpy="0 0 0" />
+      <geometry>
+        <mesh
+          filename="file://$(find cra_description)/meshes/cr30h/Link1.STL" />
+      </geometry>
+      <material
+        name="">
+        <color
+          rgba="1 1 1 1" />
+      </material>
+    </visual>
+    <collision>
+      <origin
+        xyz="0 0 0"
+        rpy="0 0 0" />
+      <geometry>
+        <mesh
+          filename="file://$(find cra_description)/meshes/cr30h/Link1.STL" />
       </geometry>
     </collision>
@@ -97,6 +97,6 @@
     type="revolute">
     <origin
-      xyz="0 0 0.23"
-      rpy="0 0 0" />
+      xyz="0 0 0.386"
+      rpy="1.5708 1.5708 0" />
     <parent
       link="base_link" />
@@ -104,5 +104,5 @@
       link="Link1" />
     <axis
-      xyz="0 0 1" />
+      xyz="-1 0 0" />
     <limit
       lower="-6.28"
@@ -115,37 +115,37 @@
     <inertial>
       <origin
-        xyz="-0.828898669983325 -3.97165169431493E-07 0.115283168336158"
-        rpy="0 0 0" />
-      <mass
-        value="0.000499668330610696" />
-      <inertia
-        ixx="0"
-        ixy="0"
-        ixz="0"
-        iyy="0"
-        iyz="0"
-        izz="0" />
-    </inertial>
-    <visual>
-      <origin
-        xyz="0 0 0"
-        rpy="0 0 0" />
-      <geometry>
-        <mesh
-          filename="file://$(find cra_description)/meshes/cr20/Link2.STL" />
-      </geometry>
-      <material
-        name="">
-        <color
-          rgba="0.792156862745098 0.819607843137255 0.933333333333333 1" />
-      </material>
-    </visual>
-    <collision>
-      <origin
-        xyz="0 0 0"
-        rpy="0 0 0" />
-      <geometry>
-        <mesh
-          filename="file://$(find cra_description)/meshes/cr20/Link2.STL" />
+        xyz="-0.398905663494017 1.92684404646904E-06 0.340471375570728"
+        rpy="0 0 0" />
+      <mass
+        value="35.1837906440538" />
+      <inertia
+        ixx="0.274172849710145"
+        ixy="-2.79808731990376E-05"
+        ixz="0.0178158997550407"
+        iyy="3.75626158130774"
+        iyz="7.44413946972762E-06"
+        izz="3.66050132171213" />
+    </inertial>
+    <visual>
+      <origin
+        xyz="0 0 0"
+        rpy="0 0 0" />
+      <geometry>
+        <mesh
+          filename="file://$(find cra_description)/meshes/cr30h/Link2.STL" />
+      </geometry>
+      <material
+        name="">
+        <color
+          rgba="1 1 1 1" />
+      </material>
+    </visual>
+    <collision>
+      <origin
+        xyz="0 0 0"
+        rpy="0 0 0" />
+      <geometry>
+        <mesh
+          filename="file://$(find cra_description)/meshes/cr30h/Link2.STL" />
       </geometry>
     </collision>
@@ -156,5 +156,5 @@
     <origin
       xyz="0 0 0"
-      rpy="1.5708 1.5708 0" />
+      rpy="0 0 0" />
     <parent
       link="Link1" />
@@ -173,37 +173,37 @@
     <inertial>
       <origin
-        xyz="-0.746000007821945 1.07337005127015E-07 0.0757301295800403"
-        rpy="0 0 0" />
-      <mass
-        value="0.00188731016390733" />
-      <inertia
-        ixx="0"
-        ixy="0"
-        ixz="0"
-        iyy="0"
-        iyz="0"
-        izz="0" />
-    </inertial>
-    <visual>
-      <origin
-        xyz="0 0 0"
-        rpy="0 0 0" />
-      <geometry>
-        <mesh
-          filename="file://$(find cra_description)/meshes/cr20/Link3.STL" />
-      </geometry>
-      <material
-        name="">
-        <color
-          rgba="0.792156862745098 0.819607843137255 0.933333333333333 1" />
-      </material>
-    </visual>
-    <collision>
-      <origin
-        xyz="0 0 0"
-        rpy="0 0 0" />
-      <geometry>
-        <mesh
-          filename="file://$(find cra_description)/meshes/cr20/Link3.STL" />
+        xyz="-0.311995849028024 -2.45961873714507E-06 0.0755143467372146"
+        rpy="0 0 0" />
+      <mass
+        value="15.319320357705" />
+      <inertia
+        ixx="0.0549431220959"
+        ixy="-7.19675342087617E-06"
+        ixz="-0.0219294614712449"
+        iyy="1.16897867168856"
+        iyz="1.09525212299586E-06"
+        izz="1.15939372786569" />
+    </inertial>
+    <visual>
+      <origin
+        xyz="0 0 0"
+        rpy="0 0 0" />
+      <geometry>
+        <mesh
+          filename="file://$(find cra_description)/meshes/cr30h/Link3.STL" />
+      </geometry>
+      <material
+        name="">
+        <color
+          rgba="1 1 1 1" />
+      </material>
+    </visual>
+    <collision>
+      <origin
+        xyz="0 0 0"
+        rpy="0 0 0" />
+      <geometry>
+        <mesh
+          filename="file://$(find cra_description)/meshes/cr30h/Link3.STL" />
       </geometry>
     </collision>
@@ -213,5 +213,5 @@
     type="revolute">
     <origin
-      xyz="-0.8252 0 0.0468"
+      xyz="-0.84 0 0"
       rpy="0 0 0" />
     <parent
@@ -220,8 +220,8 @@
       link="Link3" />
     <axis
-      xyz="0 0 1" />
-    <limit
-      lower="-2.9"
-      upper="2.9"
+      xyz="1.0869E-05 -5.499E-05 -1" />
+    <limit
+      lower="-2.79"
+      upper="2.79"
       effort="0"
       velocity="0" />
@@ -231,37 +231,37 @@
     <inertial>
       <origin
-        xyz="1.09076486456641E-07 -0.0757301256894509 1.20551504334543E-08"
-        rpy="0 0 0" />
-      <mass
-        value="0.00188731016585712" />
-      <inertia
-        ixx="0"
-        ixy="0"
-        ixz="0"
-        iyy="0"
-        iyz="0"
-        izz="0" />
-    </inertial>
-    <visual>
-      <origin
-        xyz="0 0 0"
-        rpy="0 0 0" />
-      <geometry>
-        <mesh
-          filename="file://$(find cra_description)/meshes/cr20/Link4.STL" />
-      </geometry>
-      <material
-        name="">
-        <color
-          rgba="0.792156862745098 0.819607843137255 0.933333333333333 1" />
-      </material>
-    </visual>
-    <collision>
-      <origin
-        xyz="0 0 0"
-        rpy="0 0 0" />
-      <geometry>
-        <mesh
-          filename="file://$(find cra_description)/meshes/cr20/Link4.STL" />
+        xyz="-8.57425838810129E-07 -0.0319217802585721 -0.0137198757861597"
+        rpy="0 0 0" />
+      <mass
+        value="2.61293279831353" />
+      <inertia
+        ixx="0.0104099655758254"
+        ixy="4.37316634029077E-08"
+        ixz="-1.41265169952098E-07"
+        iyy="0.00671272940307182"
+        iyz="0.00125622535616839"
+        izz="0.00920549791565436" />
+    </inertial>
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
File: cra_description/urdf/cr3_robot.xacro (robot description, xacro)
@@ -44,4 +44,5 @@
   <link  name="world"/>
 <joint name="world_joint" type="fixed">
+    <origin xyz="0 0 0.03" rpy="0 0 0" />
     <parent link="world" />
     <child  link="dummy_link" />

File: cra_description/urdf/cr5_robot.xacro (robot description, xacro)
@@ -33,4 +33,5 @@
   <link  name="world"/>
 <joint name="world_joint" type="fixed">
+    <origin xyz="0 0 0.03" rpy="0 0 0" />
     <parent link="world" />
     <child  link="dummy_link" />

File: cra_description/urdf/cr7_robot.xacro (robot description, xacro)
@@ -47,4 +47,5 @@
 <link  name="world"/>
 <joint name="world_joint" type="fixed">
+    <origin xyz="0 0 0.03" rpy="0 0 0" />
     <parent link="world" />
     <child  link="dummy_link" />

File: cra_description/urdf/me6_robot.xacro (robot description, xacro)
@@ -24,4 +24,10 @@
         </collision>
     </link>
+    <link  name="world"/>
+  <joint name="world_joint" type="fixed">
+    <origin xyz="0 0 0.03" rpy="0 0 0" />
+    <parent link="world" />
+    <child  link="dummy_link" />
+  </joint>
     <joint name="dummy_joint" type="fixed">
         <parent link="dummy_link" />

File: cra_description/urdf/nova2_robot.xacro (robot description, xacro)
@@ -3,5 +3,5 @@
     <link name="dummy_link" />
     <link name="base_link">
-<inertial>
+    <inertial>
             <origin xyz="1.31739324853774E-05 -7.84959718585273E-06 0.0647773077977383" rpy="0 0 0" />
             <mass value="0.939873286768969" />
@@ -24,4 +24,10 @@
         </collision>
     </link>
+  <link  name="world"/>
+  <joint name="world_joint" type="fixed">
+    <origin xyz="0 0 0.03" rpy="0 0 0" />
+    <parent link="world" />
+    <child  link="dummy_link" />
+  </joint>
   <joint
     name="dummy_joint"

File: cra_description/urdf/nova5_robot.xacro (robot description, xacro)
@@ -43,4 +43,10 @@
     </collision>
   </link>
+  <link  name="world"/>
+  <joint name="world_joint" type="fixed">
+    <origin xyz="0 0 0.03" rpy="0 0 0" />
+    <parent link="world" />
+    <child  link="dummy_link" />
+  </joint>
   <joint
     name="dummy_joint"

Commit message: fix cr12_gazebo_moveit

File: cra_description/urdf/cr10_robot.xacro (robot description, xacro)
@@ -2,10 +2,8 @@
 <robot name="cr10_robot" xmlns:xacro="http://ros.org/wiki/xacro">
   <link name="dummy_link"/>
-  <link
-    name="base_link">
-    <inertial>
-      <origin
-        xyz="-0.0017435 -4.7141E-06 0.032774"
-        rpy="0 0 0" />
+  <link name="base_link">
+    <inertial>
+      <origin
+        xyz="-0.0017435 -4.7141E-06 0.032774" rpy="0 0 0" />
       <mass
         value="1.8265" />

File: cra_description/urdf/cr12_robot.xacro (robot description, xacro)
@@ -1,17 +1,11 @@
 <?xml version="1.0"?>
-<!-- This URDF was automatically created by SolidWorks to URDF Exporter! Originally created by Stephen Brawner (brawner@gmail.com)
-     Commit Version: 1.6.0-1-g15f4949  Build Version: 1.6.7594.29634
-     For more information, please see http://wiki.ros.org/sw_urdf_exporter -->
 <robot
   name="cr12_robot"  xmlns:xacro="http://ros.org/wiki/xacro">
   <link name="dummy_link"/>
-  <link
-    name="base_link">
-    <inertial>
-      <origin
-        xyz="-0.00174386341900778 -4.3102660432092E-06 0.0327740188891512"
-        rpy="0 0 0" />
-      <mass
-        value="1.82652439038323" />
+  <link name="base_link">
+    <inertial>
+      <origin
+        xyz="-0.00174386341900778 -4.3102660432092E-06 0.0327740188891512" rpy="0 0 0" />
+      <mass value="1.82652439038323" />
       <inertia
         ixx="0.00417310093970523"
@@ -52,8 +46,8 @@
     <child  link="dummy_link" />
   </joint>
-     <joint name="dummy_joint" type="fixed">
+  <joint name="dummy_joint" type="fixed">
       <parent link="dummy_link" />
       <child  link="base_link" />
-    </joint>
+  </joint>
   <link
     name="Link1">

File: cra_description/urdf/cr7_robot.xacro (robot description, xacro)
@@ -1,14 +1,9 @@
 <?xml version="1.0"?>
-<!-- This URDF was automatically created by SolidWorks to URDF Exporter! Originally created by Stephen Brawner (brawner@gmail.com)
-     Commit Version: 1.6.0-1-g15f4949  Build Version: 1.6.7594.29634
-     For more information, please see http://wiki.ros.org/sw_urdf_exporter -->
 <robot name="cr7_robot"  xmlns:xacro="http://ros.org/wiki/xacro">
     <link name="dummy_link" />
-  <link
-    name="base_link">
-    <inertial>
-      <origin
-        xyz="-7.75881826404344E-06 0.00191109737802069 0.0289949710713939"
-        rpy="0 0 0" />
+  <link name="base_link">
+    <inertial>
+      <origin
+        xyz="-7.75881826404344E-06 0.00191109737802069 0.0289949710713939" rpy="0 0 0" />
       <mass
         value="0.908795453638862" />
