Commit message: update CR3A/CR5A URDF

File: cra_description/urdf/cr3_robot.xacro (robot description, xacro)
@@ -6,15 +6,15 @@
     <inertial>
       <origin
-        xyz="-0.0027213 3.915E-07 0.022038"
-        rpy="0 0 0" />
-      <mass
-        value="0.653" />
-      <inertia
-        ixx="0.00075137"
-        ixy="-3.0366E-08"
-        ixz="1.2825E-06"
-        iyy="0.00080094"
-        iyz="2.5423E-09"
-        izz="0.0010902" />
+        xyz="0.00230818905212046 -0.000732843557555838 0.028289656612971"
+        rpy="0 0 0" />
+      <mass
+        value="0.648931294984644" />
+      <inertia
+        ixx="0.000749921651777976"
+        ixy="4.21801992495725E-08"
+        ixz="1.27081371753695E-06"
+        iyy="0.000839640950438419"
+        iyz="1.61611917342073E-07"
+        izz="0.00112778981497252" />
     </inertial>
     <visual>
@@ -29,5 +29,5 @@
         name="">
         <color
-          rgba="1 1 1 1" />
+          rgba="0.792156862745098 0.819607843137255 0.933333333333333 1" />
       </material>
     </visual>
@@ -43,5 +43,5 @@
   </link>
   <link  name="world"/>
-<joint name="world_joint" type="fixed">
+  <joint name="world_joint" type="fixed">
     <origin xyz="0 0 0.03" rpy="0 0 0" />
     <parent link="world" />
@@ -49,44 +49,44 @@
   </joint>
   <joint name="dummy_joint" type="fixed">
-    <parent link="dummy_link" />
-    <child  link="base_link" />
-  </joint>
+      <parent link="dummy_link" />
+      <child  link="base_link" />
+    </joint>
   <link
     name="Link1">
     <inertial>
       <origin
-        xyz="-3.68657602416735E-05 -0.00394516685385322 0.00364037839421286"
-        rpy="0 0 0" />
-      <mass
-        value="1.31100598822002" />
-      <inertia
-        ixx="0.00202531167977736"
-        ixy="-1.62039964254407E-06"
-        ixz="4.44242218921916E-07"
-        iyy="0.00198085794611413"
-        iyz="0.000256891817572315"
-        izz="0.00183966900872187" />
-    </inertial>
-    <visual>
-      <origin
-        xyz="0 0 0"
-        rpy="0 0 0" />
-      <geometry>
-        <mesh
-          filename="file://$(find cra_description)/meshes/cr3/Link1.STL" />
-      </geometry>
-      <material
-        name="">
-        <color
-          rgba="1 1 1 1" />
-      </material>
-    </visual>
-    <collision>
-      <origin
-        xyz="0 0 0"
-        rpy="0 0 0" />
-      <geometry>
-        <mesh
-          filename="file://$(find cra_description)/meshes/cr3/Link1.STL" />
+        xyz="-3.67781721123111E-05 -0.00394376486631129 0.00364267890020981"
+        rpy="0 0 0" />
+      <mass
+        value="1.31115064359517" />
+      <inertia
+        ixx="0.00319192385509536"
+        ixy="-1.81661180744991E-06"
+        ixz="-3.59316770697547E-07"
+        iyy="0.00307821666880085"
+        iyz="-1.88925967107205E-05"
+        izz="0.00190896903282013" />
+    </inertial>
+    <visual>
+      <origin
+        xyz="0 0 0"
+        rpy="0 0 0" />
+      <geometry>
+        <mesh
+          filename="file://$(find cra_description)/meshes/cr3/J1.STL" />
+      </geometry>
+      <material
+        name="">
+        <color
+          rgba="0.792156862745098 0.819607843137255 0.933333333333333 1" />
+      </material>
+    </visual>
+    <collision>
+      <origin
+        xyz="0 0 0"
+        rpy="0 0 0" />
+      <geometry>
+        <mesh
+          filename="file://$(find cra_description)/meshes/cr3/J1.STL" />
       </geometry>
     </collision>
@@ -96,6 +96,6 @@
     type="revolute">
     <origin
-      xyz="0 0 0.1283"
-      rpy="0 0 0" />
+      xyz="0 0 0.1348"
+      rpy="0 0 -1.5708" />
     <parent
       link="base_link" />
@@ -105,8 +105,8 @@
       xyz="0 0 1" />
     <limit
-      lower="-6.27"
-      upper="6.27"
-      effort="300"
-      velocity="100" />
+      lower="-6.28"
+      upper="6.28"
+      effort="0"
+      velocity="0" />
   </joint>
   <link
@@ -114,37 +114,37 @@
     <inertial>
       <origin
-        xyz="-0.129235280055448 1.440541622715E-05 0.133173619961293"
-        rpy="0 0 0" />
-      <mass
-        value="3.40043726977504" />
-      <inertia
-        ixx="0.00450581324845612"
-        ixy="1.58054368766225E-06"
-        ixz="8.56287041890268E-05"
-        iyy="0.00632329822349442"
-        iyz="-4.41201729949356E-07"
-        izz="0.00578241711656701" />
-    </inertial>
-    <visual>
-      <origin
-        xyz="0 0 0"
-        rpy="0 0 0" />
-      <geometry>
-        <mesh
-          filename="file://$(find cra_description)/meshes/cr3/Link2.STL" />
-      </geometry>
-      <material
-        name="">
-        <color
-          rgba="1 1 1 1" />
-      </material>
-    </visual>
-    <collision>
-      <origin
-        xyz="0 0 0"
-        rpy="0 0 0" />
-      <geometry>
-        <mesh
-          filename="file://$(find cra_description)/meshes/cr3/Link2.STL" />
+        xyz="-0.129228226099202 1.43480420269969E-05 0.133174339594273"
+        rpy="0 0 0" />
+      <mass
+        value="3.40049600294342" />
+      <inertia
+        ixx="0.00665284748175434"
+        ixy="1.79448081220597E-06"
+        ixz="0.000635378334498705"
+        iyy="0.0177342976210456"
+        iyz="3.48633745916203E-07"
+        izz="0.0150462633110018" />
+    </inertial>
+    <visual>
+      <origin
+        xyz="0 0 0"
+        rpy="0 0 0" />
+      <geometry>
+        <mesh
+          filename="file://$(find cra_description)/meshes/cr3/J2.STL" />
+      </geometry>
+      <material
+        name="">
+        <color
+          rgba="0.792156862745098 0.819607843137255 0.933333333333333 1" />
+      </material>
+    </visual>
+    <collision>
+      <origin
+        xyz="0 0 0"
+        rpy="0 0 0" />
+      <geometry>
+        <mesh
+          filename="file://$(find cra_description)/meshes/cr3/J2.STL" />
       </geometry>
     </collision>
@@ -163,8 +163,8 @@
       xyz="0 0 1" />
     <limit
-      lower="-6.27"
-      upper="6.27"
-      effort="300"
-      velocity="100" />
+      lower="-6.28"
+      upper="6.28"
+      effort="0"
+      velocity="0" />
   </joint>
   <link
@@ -172,37 +172,37 @@
     <inertial>
       <origin
-        xyz="-0.119822632176479 8.63344146663093E-08 0.0099876637825216"
-        rpy="0 0 0" />
-      <mass
-        value="2.21449412948544" />
-      <inertia
-        ixx="0.00236120280734313"
-        ixy="1.81888962826726E-08"
-        ixz="0.000137629457194959"
-        iyy="0.00313635345351584"
-        iyz="-1.39166877342495E-08"
-        izz="0.00285118872456311" />
-    </inertial>
-    <visual>
-      <origin
-        xyz="0 0 0"
-        rpy="0 0 0" />
-      <geometry>
-        <mesh
-          filename="file://$(find cra_description)/meshes/cr3/Link3.STL" />
-      </geometry>
-      <material
-        name="">
-        <color
-          rgba="1 1 1 1" />
-      </material>
-    </visual>
-    <collision>
-      <origin
-        xyz="0 0 0"
-        rpy="0 0 0" />
-      <geometry>
-        <mesh
-          filename="file://$(find cra_description)/meshes/cr3/Link3.STL" />
+        xyz="-0.121267841067619 -5.95979094526938E-07 0.0103431444175778"
+        rpy="0 0 0" />
+      <mass
+        value="2.18803928124499" />
+      <inertia
+        ixx="0.0031393454782363"
+        ixy="2.60060285754048E-07"
+        ixz="-0.000151120131479005"
+        iyy="0.0236694689770697"
+        iyz="3.67396297009222E-08"
+        izz="0.0225795743545604" />
+    </inertial>
+    <visual>
+      <origin
+        xyz="0 0 0"
+        rpy="0 0 0" />
+      <geometry>
+        <mesh
+          filename="file://$(find cra_description)/meshes/cr3/J3.STL" />
+      </geometry>
+      <material
+        name="">
+        <color
+          rgba="0.792156862745098 0.819607843137255 0.933333333333333 1" />
+      </material>
+    </visual>
+    <collision>
+      <origin
+        xyz="0 0 0"
+        rpy="0 0 0" />
+      <geometry>
+        <mesh
+          filename="file://$(find cra_description)/meshes/cr3/J3.STL" />
       </geometry>
     </collision>
@@ -221,8 +221,8 @@
       xyz="0 0 1" />
     <limit
-      lower="-2.86"
-      upper="2.86"
-      effort="300"
-      velocity="100" />
+      lower="-2.7039"
+      upper="2.7039"
+      effort="0"
+      velocity="0" />
   </joint>
   <link
@@ -230,37 +230,37 @@
     <inertial>
       <origin
-        xyz="1.74679534498573E-07 0.0034522361215461 -0.0028730999658578"
-        rpy="0 0 0" />
-      <mass
-        value="0.842272956366123" />
-      <inertia
-        ixx="0.00100389823526424"
-        ixy="-3.26498724132116E-09"
-        ixz="-3.83652674720848E-09"
-        iyy="0.000793473566890046"
-        iyz="0.000133420135294005"
-        izz="0.000993889852029541" />
-    </inertial>
-    <visual>
-      <origin
-        xyz="0 0 0"
-        rpy="0 0 0" />
-      <geometry>
-        <mesh
-          filename="file://$(find cra_description)/meshes/cr3/Link4.STL" />
-      </geometry>
-      <material
-        name="">
-        <color
-          rgba="1 1 1 1" />
-      </material>
-    </visual>
-    <collision>
-      <origin
-        xyz="0 0 0"
-        rpy="0 0 0" />
-      <geometry>
-        <mesh
-          filename="file://$(find cra_description)/meshes/cr3/Link4.STL" />
+        xyz="1.66290133222139E-07 0.00345100795834197 -0.00287330777509653"
+        rpy="0 0 0" />
+      <mass
+        value="0.842219175919104" />
+      <inertia
+        ixx="0.00173365879213697"
+        ixy="-4.56469972647882E-09"
+        ixz="-4.71044121344451E-10"
+        iyy="0.000822485798327018"
+        iyz="-9.31644060918737E-06"
+        izz="0.00169454892249307" />
+    </inertial>
+    <visual>
+      <origin
+        xyz="0 0 0"
+        rpy="0 0 0" />
+      <geometry>
+        <mesh
+          filename="file://$(find cra_description)/meshes/cr3/J4.STL" />
+      </geometry>
+      <material
+        name="">
+        <color
+          rgba="0.792156862745098 0.819607843137255 0.933333333333333 1" />
+      </material>
+    </visual>
+    <collision>
+      <origin
+        xyz="0 0 0"
+        rpy="0 0 0" />
+      <geometry>
+        <mesh
+          filename="file://$(find cra_description)/meshes/cr3/J4.STL" />
       </geometry>
     </collision>
@@ -268,5 +268,5 @@
   <joint
     name="joint4"
-    type="revolute">
+    type="continuous">
     <origin
       xyz="-0.23 0 0.1283"
@@ -277,10 +277,10 @@
       link="Link4" />
     <axis
-      xyz="0 0 1" />
+      xyz="0 0 -1" />
     <limit
-      lower="-6.27"
-      upper="6.27"
-      effort="300"
-      velocity="100" />
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
File: cra_description/urdf/cr5_robot.xacro (robot description, xacro)
@@ -1,36 +1,47 @@
 <?xml version="1.0"?>
 <robot name="cr5_robot" xmlns:xacro="http://ros.org/wiki/xacro">
- <link name="dummy_link" />
- <link name="base_link">
-    <inertial>
-      <origin xyz="-8.0961E-06 0.0019103 0.028995" rpy="0 0 0" />
-      <mass value="0.90882" />
-      <inertia
-        ixx="0"
-        ixy="0"
-        ixz="0"
-        iyy="0"
-        iyz="0"
-        izz="0" />
-    </inertial>
-    <visual>
-      <origin xyz="0 0 0" rpy="0 0 0" />
-      <geometry>
-        <mesh filename="file://$(find cra_description)/meshes/cr5/base_link.dae" />
-      </geometry>
-      <material
-        name="">
-        <color rgba="0 0 0 1" />
-      </material>
-    </visual>
-    <collision>
-      <origin xyz="0 0 0" rpy="0 0 0" />
-      <geometry>
-        <mesh filename="file://$(find cra_description)/meshes/cr5/base_link.dae" />
+  <link name="dummy_link" />
+  <link
+    name="base_link">
+    <inertial>
+      <origin
+        xyz="-7.94481692926771E-06 0.00312979848669993 0.0289305341801692"
+        rpy="0 0 0" />
+      <mass
+        value="0.921803441591401" />
+      <inertia
+        ixx="0.00155218443258025"
+        ixy="4.57972945608826E-08"
+        ixz="-1.88985548171397E-07"
+        iyy="0.0013468290665964"
+        iyz="-1.49049888586631E-06"
+        izz="0.00225259728822295" />
+    </inertial>
+    <visual>
+      <origin
+        xyz="0 0 0"
+        rpy="0 0 0" />
+      <geometry>
+        <mesh
+          filename="file://$(find cra_description)/meshes/cr5/base_link.STL" />
+      </geometry>
+      <material
+        name="">
+        <color
+          rgba="0.792156862745098 0.819607843137255 0.933333333333333 1" />
+      </material>
+    </visual>
+    <collision>
+      <origin
+        xyz="0 0 0"
+        rpy="0 0 0" />
+      <geometry>
+        <mesh
+          filename="file://$(find cra_description)/meshes/cr5/base_link.STL" />
       </geometry>
     </collision>
   </link>
   <link  name="world"/>
-<joint name="world_joint" type="fixed">
+  <joint name="world_joint" type="fixed">
     <origin xyz="0 0 0.03" rpy="0 0 0" />
     <parent link="world" />
@@ -38,220 +49,354 @@
   </joint>
   <joint name="dummy_joint" type="fixed">
-    <parent link="dummy_link" />
-    <child  link="base_link" />
-  </joint>
-  <link  name="Link1">
-    <inertial>
-      <origin xyz="-8.7268E-07 -0.0032576 -0.0076748" rpy="0 0 0" />
-      <mass value="1.6123" />
-      <inertia
-        ixx="0"
-        ixy="0"
-        ixz="0"
-        iyy="0"
-        iyz="0"
-        izz="0" />
-    </inertial>
-    <visual>
-      <origin xyz="0 0 0" rpy="0 0 0" />
-      <geometry>
-        <mesh filename="file://$(find cra_description)/meshes/cr5/Link1.dae" />
-      </geometry>
-      <material
-        name="">
-        <color rgba="1 1 1 1" />
-      </material>
-    </visual>
-    <collision>
-      <origin xyz="0 0 0" rpy="0 0 0" />
-      <geometry>
-        <mesh filename="file://$(find cra_description)/meshes/cr5/Link1.dae" />
-      </geometry>
-    </collision>
-  </link>
-  <joint name="joint1" type="revolute">
-    <origin xyz="0 0 0.147" rpy="0 0 0" />
-    <parent link="base_link" />
-    <child link="Link1" />
-    <axis xyz="0 0 1" />
-    <limit lower="-6.27" upper="6.27" effort="300" velocity="100" />
-  </joint>
-  <link name="Link2">
-    <inertial>
-      <origin xyz="-0.21351 -1.3842E-06 0.14252" rpy="0 0 0" />
-      <mass value="5.5186" />
-      <inertia
-        ixx="0"
-        ixy="0"
-        ixz="0"
-        iyy="0"
-        iyz="0"
-        izz="0" />
-    </inertial>
-    <visual>
-      <origin xyz="0 0 0" rpy="0 0 0" />
-      <geometry>
-         <mesh filename="file://$(find cra_description)/meshes/cr5/Link2.dae" />
-      </geometry>
-      <material
-        name="">
-        <color rgba="1 1 1 1" />
-      </material>
-    </visual>
-    <collision>
-      <origin xyz="0 0 0" rpy="0 0 0" />
-      <geometry>
-        <mesh filename="file://$(find cra_description)/meshes/cr5/Link2.dae" />
-      </geometry>
-    </collision>
-  </link>
-  <joint name="joint2" type="revolute">
-    <origin xyz="0 0 0" rpy="1.5708 1.5708 0" />
-    <parent link="Link1" />
-    <child  link="Link2" />
-    <axis xyz="0 0 1" />
-    <limit lower="-6.27" upper="6.27" effort="300" velocity="100" />
-  </joint>
-  <link name="Link3">
-    <inertial>
-      <origin xyz="-0.15231 -1.4079E-07 0.022693" rpy="0 0 0" />
-      <mass value="2.8536" />
-      <inertia
-        ixx="0"
-        ixy="0"
-        ixz="0"
-        iyy="0"
-        iyz="0"
-        izz="0" />
-    </inertial>
-    <visual>
-      <origin xyz="0 0 0" rpy="0 0 0" />
-      <geometry>
-        <mesh filename="file://$(find cra_description)/meshes/cr5/Link3.dae" />
-      </geometry>
-      <material
-        name="">
-        <color rgba="1 1 1 1" />
-      </material>
-    </visual>
-    <collision>
-      <origin xyz="0 0 0"  rpy="0 0 0" />
-      <geometry>
-        <mesh filename="file://$(find cra_description)/meshes/cr5/Link3.dae" />
-      </geometry>
-    </collision>
-  </link>
-  <joint name="joint3" type="revolute">
-    <origin xyz="-0.427 0 0" rpy="0 0 0" />
-    <parent link="Link2" />
-    <child link="Link3" />
-    <axis  xyz="0 0 1" />
-    <limit lower="-2.86"  upper="2.86"  effort="300" velocity="100" />
-  </joint>
-  <link name="Link4">
-    <inertial>
-      <origin xyz="-3.2386E-07 -0.002077 -0.0015548" rpy="0 0 0" />
-      <mass value="0.67058" />
-      <inertia
-        ixx="0"
-        ixy="0"
-        ixz="0"
-        iyy="0"
-        iyz="0"
-        izz="0" />
-    </inertial>
-    <visual>
-      <origin xyz="0 0 0" rpy="0 0 0" />
-      <geometry>
-        <mesh filename="file://$(find cra_description)/meshes/cr5/Link4.dae" />
-      </geometry>
-      <material name="">
-        <color rgba="1 1 1 1" />
-      </material>
-    </visual>
-    <collision>
-      <origin xyz="0 0 0" rpy="0 0 0" />
-      <geometry>
-        <mesh filename="file://$(find cra_description)/meshes/cr5/Link4.dae" />
-      </geometry>
-    </collision>
-  </link>
-  <joint name="joint4" type="revolute">
-    <origin xyz="-0.357 0 0.141" rpy="0 0 -1.5708" />
-    <parent link="Link3" />
-    <child link="Link4" />
-    <axis xyz="0 0 1" />
-    <limit lower="-6.27" upper="6.27" effort="300" velocity="100" />
+      <parent link="dummy_link" />
+      <child  link="base_link" />
+    </joint>
+  <link
+    name="Link1">
+    <inertial>
+      <origin
+        xyz="1.73246183103459E-07 -0.00325457191611467 -0.00763347019440543"
+        rpy="0 0 0" />
+      <mass
+        value="1.61309076753593" />
+      <inertia
+        ixx="0.00546783618974324"
+        ixy="1.55105105896333E-09"
+        ixz="-7.41656921043421E-08"
+        iyy="0.00525034621721433"
+        iyz="-9.78846785618848E-05"
+        izz="0.00340956817185818" />
+    </inertial>
+    <visual>
+      <origin
+        xyz="0 0 0"
+        rpy="0 0 0" />
+      <geometry>
+        <mesh
+          filename="file://$(find cra_description)/meshes/cr5/J1.STL" />
+      </geometry>
+      <material
+        name="">
+        <color
+          rgba="0.792156862745098 0.819607843137255 0.933333333333333 1" />
+      </material>
+    </visual>
+    <collision>
+      <origin
+        xyz="0 0 0"
+        rpy="0 0 0" />
+      <geometry>
+        <mesh
+          filename="file://$(find cra_description)/meshes/cr5/J1.STL" />
+      </geometry>
+    </collision>
+  </link>
+  <joint
+    name="joint1"
+    type="revolute">
+    <origin
+      xyz="0 0 0.147"
+      rpy="0 0 0" />
+    <parent
+      link="base_link" />
+    <child
+      link="Link1" />
+    <axis
+      xyz="0 0 1" />
+    <limit
+      lower="-6.28"
+      upper="6.28"
+      effort="0"
+      velocity="0" />
+  </joint>
+  <link
+    name="Link2">
+    <inertial>
+      <origin
+        xyz="-0.213514541447242 -0.000174145825908622 0.142532293229243"
+        rpy="0 0 0" />
+      <mass
+        value="5.52502766431306" />
+      <inertia
+        ixx="0.0135390102321012"
+        ixy="-0.000132792191512557"
+        ixz="1.08942594671362E-06"
+        iyy="0.175351190928579"
+        iyz="-1.55761894405212E-07"
+        izz="0.171155665794094" />
+    </inertial>
+    <visual>
+      <origin
+        xyz="0 0 0"
+        rpy="0 0 0" />
+      <geometry>
+        <mesh
+          filename="file://$(find cra_description)/meshes/cr5/J2.STL" />
+      </geometry>
+      <material
+        name="">
+        <color
+          rgba="0.792156862745098 0.819607843137255 0.933333333333333 1" />
+      </material>
+    </visual>
+    <collision>
+      <origin
+        xyz="0 0 0"
+        rpy="0 0 0" />
+      <geometry>
+        <mesh
+          filename="file://$(find cra_description)/meshes/cr5/J2.STL" />
+      </geometry>
+    </collision>
+  </link>
+  <joint
+    name="joint2"
+    type="revolute">
+    <origin
+      xyz="0 0 0"
+      rpy="1.5708 1.5708 0" />
+    <parent
+      link="Link1" />
+    <child
+      link="Link2" />
+    <axis
+      xyz="0 0 1" />
+    <limit
+      lower="-6.28"
+      upper="6.28"
+      effort="0"
+      velocity="0" />
+  </joint>
+  <link
+    name="Link3">
+    <inertial>
+      <origin
+        xyz="-0.152341668261688 0.000149359452503151 0.0226831470311876"
+        rpy="0 0 0" />
+      <mass
+        value="2.85389421082174" />
+      <inertia
+        ixx="0.00426233866492008"
+        ixy="5.97680353890416E-05"
+        ixz="0.00145366515031237"
+        iyy="0.0651295114823361"
+        iyz="-1.39806459057094E-06"
+        izz="0.0643864464792015" />
+    </inertial>
+    <visual>
+      <origin
+        xyz="0 0 0"
+        rpy="0 0 0" />
+      <geometry>
+        <mesh
+          filename="file://$(find cra_description)/meshes/cr5/J3.STL" />
+      </geometry>
+      <material
+        name="">
+        <color
+          rgba="0.792156862745098 0.819607843137255 0.933333333333333 1" />
+      </material>
+    </visual>
+    <collision>
+      <origin
+        xyz="0 0 0"
+        rpy="0 0 0" />
+      <geometry>
+        <mesh
+          filename="file://$(find cra_description)/meshes/cr5/J3.STL" />
+      </geometry>
+    </collision>
+  </link>
+  <joint
+    name="joint3"
+    type="revolute">
+    <origin
+      xyz="-0.427 -0.00034866 0"
+      rpy="0 0 0" />
+    <parent
+      link="Link2" />
+    <child
+      link="Link3" />
+    <axis
+      xyz="0 0 1" />
+    <limit
+      lower="-2.792"
+      upper="2.792"
+      effort="0"
+      velocity="0" />
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