Commit message: update CR3A/CR5A URDF

File: dobot_rviz/urdf/cr3_robot.urdf (robot description, URDF)
Before this commit: robot cr3_robot, 8 links, 7 joints
Links:
- link Link1: mass 1.31100598822002 -> 1.31115064359517; geometry collision mesh filename=package://dobot_rviz/meshes/cr3/J1.STL; visual mesh filename=package://dobot_rviz/meshes/cr3/J1.STL
- link Link2: mass 3.40043726977504 -> 3.40049600294342; geometry collision mesh filename=package://dobot_rviz/meshes/cr3/J2.STL; visual mesh filename=package://dobot_rviz/meshes/cr3/J2.STL
- link Link3: mass 2.21449412948544 -> 2.18803928124499; geometry collision mesh filename=package://dobot_rviz/meshes/cr3/J3.STL; visual mesh filename=package://dobot_rviz/meshes/cr3/J3.STL
- link Link4: mass 0.842272956366123 -> 0.842219175919104; geometry collision mesh filename=package://dobot_rviz/meshes/cr3/J4.STL; visual mesh filename=package://dobot_rviz/meshes/cr3/J4.STL
- link Link5: mass 0.843692877114241 -> 0.741136954868999; geometry collision mesh filename=package://dobot_rviz/meshes/cr3/J5.STL; visual mesh filename=package://dobot_rviz/meshes/cr3/J5.STL
- link Link6: mass 0.159409278145106 -> 0.157885369717385; geometry collision mesh filename=package://dobot_rviz/meshes/cr3/J6.STL; visual mesh filename=package://dobot_rviz/meshes/cr3/J6.STL
- link base_link: mass 0.653 -> 0.648931294984644
Joints:
- joint joint1: limit lower=-6.27 upper=6.27 effort=0 velocity=0 -> lower=-6.28 upper=6.28 effort=0 velocity=0; origin xyz=0 0 0.1283 rpy=0 0 0 -> xyz=0 0 0.1348 rpy=0 0 -1.5708
- joint joint2: limit lower=-6.27 upper=6.27 effort=0 velocity=0 -> lower=-6.28 upper=6.28 effort=0 velocity=0
- joint joint3: limit lower=-2.86 upper=2.86 effort=0 velocity=0 -> lower=-2.7039 upper=2.7039 effort=0 velocity=0
- joint joint4: axis 0 0 1 -> 0 0 -1; limit lower=-6.27 upper=6.27 effort=0 velocity=0 -> lower=-6.28 upper=6.28 effort=0 velocity=0; type revolute -> continuous
- joint joint5: axis 0 0 1 -> 0 0 -1; limit lower=-6.27 upper=6.27 effort=0 velocity=0 -> lower=-6.28 upper=6.28 effort=0 velocity=0; type revolute -> continuous
- joint joint6: axis 0 0 1 -> 0 0 -1; limit lower=-6.27 upper=6.27 effort=0 velocity=0 -> lower=-6.28 upper=6.28 effort=0 velocity=0

File: dobot_rviz/urdf/cr5_robot.urdf (robot description, URDF)
Before this commit: robot cr5_robot, 8 links, 7 joints
Links:
- link Link1: mass 1.6123 -> 1.61309076753593; geometry collision mesh filename=package://dobot_rviz/meshes/cr5/J1.STL; visual mesh filename=package://dobot_rviz/meshes/cr5/J1.STL
- link Link2: mass 5.5186 -> 5.52502766431306; geometry collision mesh filename=package://dobot_rviz/meshes/cr5/J2.STL; visual mesh filename=package://dobot_rviz/meshes/cr5/J2.STL
- link Link3: mass 2.8536 -> 2.85389421082174; geometry collision mesh filename=package://dobot_rviz/meshes/cr5/J3.STL; visual mesh filename=package://dobot_rviz/meshes/cr5/J3.STL
- link Link4: mass 0.67058 -> 0.670967728058518; geometry collision mesh filename=package://dobot_rviz/meshes/cr5/J4.STL; visual mesh filename=package://dobot_rviz/meshes/cr5/J4.STL
- link Link5: mass 0.7269 -> 0.741136954745254; geometry collision mesh filename=package://dobot_rviz/meshes/cr5/J5.STL; visual mesh filename=package://dobot_rviz/meshes/cr5/J5.STL
- link Link6: mass 0.15789 -> 0.157885369717385; geometry collision mesh filename=package://dobot_rviz/meshes/cr5/J6.STL; visual mesh filename=package://dobot_rviz/meshes/cr5/J6.STL
- link base_link: mass 0.90882 -> 0.921803441591401; geometry collision mesh filename=package://dobot_rviz/meshes/cr5/base_link.STL; visual mesh filename=package://dobot_rviz/meshes/cr5/base_link.STL
Joints:
- joint joint1: limit lower=-6.27 upper=6.27 effort=0 velocity=0 -> lower=-6.28 upper=6.28 effort=0 velocity=0
- joint joint2: limit lower=-6.27 upper=6.27 effort=0 velocity=0 -> lower=-6.28 upper=6.28 effort=0 velocity=0
- joint joint3: limit lower=-2.86 upper=2.86 effort=0 velocity=0 -> lower=-2.792 upper=2.792 effort=0 velocity=0; origin xyz=-0.427 0 0 rpy=0 0 0 -> xyz=-0.427 -0.00034866 0 rpy=0 0 0
- joint joint4: limit lower=-6.27 upper=6.27 effort=0 velocity=0 -> lower=-6.28 upper=6.28 effort=0 velocity=0; origin xyz=-0.357 0 0.141 rpy=0 0 -1.5708 -> xyz=-0.357 0.00034866 0.141 rpy=0 0 -1.5708
- joint joint5: limit lower=-6.27 upper=6.27 effort=0 velocity=0 -> lower=-6.28 upper=6.28 effort=0 velocity=0
- joint joint6: limit lower=-6.27 upper=6.27 effort=0 velocity=0 -> lower=-6.28 upper=6.28 effort=0 velocity=0
