Commit message: update nova5-xacro

File: cra_description/urdf/nova5_robot.xacro (robot description, xacro)
@@ -45,5 +45,4 @@
   <link  name="world"/>
   <joint name="world_joint" type="fixed">
-    <origin xyz="0 0 0.03" rpy="0 0 0" />
     <parent link="world" />
     <child  link="dummy_link" />
@@ -108,10 +107,10 @@
       link="Link1" />
     <axis
-      xyz="0 0 -0.999999999999855" />
+      xyz="0 0 0.999999999999855" />
     <limit
       lower="-6.28"
       upper="6.28"
-      effort="300"
-      velocity="100" />
+      effort="0"
+      velocity="0" />
   </joint>
   <link
@@ -170,6 +169,6 @@
       lower="-3.14"
       upper="3.14"
-      effort="300"
-      velocity="100" />
+      effort="0"
+      velocity="0" />
   </joint>
   <link
@@ -228,6 +227,6 @@
       lower="-2.79"
       upper="2.79"
-      effort="300"
-      velocity="100" />
+      effort="0"
+      velocity="0" />
   </joint>
   <link
@@ -282,10 +281,10 @@
       link="Link4" />
     <axis
-      xyz="0 0 -1" />
+      xyz="0 0 1" />
     <limit
       lower="-6.28"
       upper="6.28"
-      effort="300"
-      velocity="100" />
+      effort="0"
+      velocity="0" />
   </joint>
   <link
@@ -344,6 +343,6 @@
       lower="-6.28"
       upper="6.28"
-      effort="300"
-      velocity="100" />
+      effort="0"
+      velocity="0" />
   </joint>
   <link
@@ -402,6 +401,6 @@
       lower="-6.28"
       upper="6.28"
-      effort="300"
-      velocity="100" />
+      effort="0"
+      velocity="0" />
   </joint>
    <gazebo reference="base_link">
