Commit message: fix: correct orientation direction of URDF model

File: cra_description/urdf/cr10af_robot.xacro (robot description, xacro)
@@ -53,5 +53,5 @@
     </joint>
   <link
-    name="J1">
+    name="Link1">
     <inertial>
       <origin
@@ -101,5 +101,5 @@
       link="base_link" />
     <child
-      link="J1" />
+      link="Link1" />
     <axis
       xyz="0 0 1" />
@@ -111,5 +111,5 @@
   </joint>
   <link
-    name="J2">
+    name="Link2">
     <inertial>
       <origin
@@ -157,7 +157,7 @@
       rpy="0 0 0" />
     <parent
-      link="J1" />
+      link="Link1" />
     <child
-      link="J2" />
+      link="Link2" />
     <axis
       xyz="0 -1 0" />
@@ -169,5 +169,5 @@
   </joint>
   <link
-    name="J3">
+    name="Link3">
     <inertial>
       <origin
@@ -215,9 +215,9 @@
       rpy="0 0 0" />
     <parent
-      link="J2" />
+      link="Link2" />
     <child
-      link="J3" />
+      link="Link3" />
     <axis
-      xyz="0 1 0" />
+      xyz="0 -1 0" />
     <limit
       lower="-2.7925"
@@ -227,5 +227,5 @@
   </joint>
   <link
-    name="J4">
+    name="Link4">
     <inertial>
       <origin
@@ -273,7 +273,7 @@
       rpy="0 0 0" />
     <parent
-      link="J3" />
+      link="Link3" />
     <child
-      link="J4" />
+      link="Link4" />
     <axis
       xyz="0 -1 0" />
@@ -285,5 +285,5 @@
   </joint>
   <link
-    name="J5">
+    name="Link5">
     <inertial>
       <origin
@@ -331,7 +331,7 @@
       rpy="0 0 0" />
     <parent
-      link="J4" />
+      link="Link4" />
     <child
-      link="J5" />
+      link="Link5" />
     <axis
       xyz="0 0 1" />
@@ -343,5 +343,5 @@
   </joint>
   <link
-    name="J6">
+    name="Link6">
     <inertial>
       <origin
@@ -389,7 +389,7 @@
       rpy="0 0 0" />
     <parent
-      link="J5" />
+      link="Link5" />
     <child
-      link="J6" />
+      link="Link6" />
     <axis
       xyz="0 -1 0" />
@@ -400,29 +400,35 @@
       velocity="0" />
   </joint>
+  <link name="tool0"/>
+  <joint name="tool_joint" type="fixed">
+    <origin xyz="0 0 0" rpy="4.7124 0 3.14159" />
+    <parent link="Link6" />
+    <child link="tool0" />
+  </joint>
 <gazebo reference="base_link">
         <gravity>false</gravity>
         <selfCollide>true</selfCollide>
     </gazebo>
-    <gazebo reference="Link1">
-        <gravity>false</gravity>
-        <selfCollide>true</selfCollide>
-    </gazebo>
-    <gazebo reference="Link2">
-        <gravity>false</gravity>
-        <selfCollide>true</selfCollide>
-    </gazebo>
-    <gazebo reference="Link3">
-        <gravity>false</gravity>
-        <selfCollide>true</selfCollide>
-    </gazebo>
-    <gazebo reference="Link4">
-        <gravity>false</gravity>
-        <selfCollide>true</selfCollide>
-    </gazebo>
-    <gazebo reference="Link5">
-        <gravity>false</gravity>
-        <selfCollide>true</selfCollide>
-    </gazebo>
-    <gazebo reference="Link6">
+    <gazebo reference="J1">
+        <gravity>false</gravity>
+        <selfCollide>true</selfCollide>
+    </gazebo>
+    <gazebo reference="J2">
+        <gravity>false</gravity>
+        <selfCollide>true</selfCollide>
+    </gazebo>
+    <gazebo reference="J3">
+        <gravity>false</gravity>
+        <selfCollide>true</selfCollide>
+    </gazebo>
+    <gazebo reference="J4">
+        <gravity>false</gravity>
+        <selfCollide>true</selfCollide>
+    </gazebo>
+    <gazebo reference="J5">
+        <gravity>false</gravity>
+        <selfCollide>true</selfCollide>
+    </gazebo>
+    <gazebo reference="J6">
         <gravity>false</gravity>
         <selfCollide>true</selfCollide>

File: cra_description/urdf/cr30h_robot.xacro (robot description, xacro)
@@ -98,5 +98,5 @@
     <origin
       xyz="0 0 0.386"
-      rpy="1.5708 1.5708 0" />
+      rpy="0 0 0" />
     <parent
       link="base_link" />
@@ -104,5 +104,5 @@
       link="Link1" />
     <axis
-      xyz="-1 0 0" />
+      xyz="0 0 1" />
     <limit
       lower="-6.28"
@@ -394,5 +394,5 @@
       link="Link6" />
     <axis
-      xyz="0 0 -1" />
+      xyz="0 0 1" />
     <limit
       lower="-6.28"

File: cra_description/urdf/cr3_robot.xacro (robot description, xacro)
@@ -97,5 +97,5 @@
     <origin
       xyz="0 0 0.1348"
-      rpy="0 0 -1.5708" />
+      rpy="0 0 0" />
     <parent
       link="base_link" />
@@ -268,5 +268,5 @@
   <joint
     name="joint4"
-    type="continuous">
+    type="revolute">
     <origin
       xyz="-0.23 0 0.1283"
@@ -277,5 +277,5 @@
       link="Link4" />
     <axis
-      xyz="0 0 -1" />
+      xyz="0 0 1" />
     <limit
       lower="-6.28"
@@ -326,5 +326,5 @@
   <joint
     name="joint5"
-    type="continuous">
+    type="revolute">
     <origin
       xyz="0 -0.116 0"
@@ -335,5 +335,5 @@
       link="Link5" />
     <axis
-      xyz="0 0 -1" />
+      xyz="0 0 1" />
     <limit
       lower="-6.28"
@@ -393,5 +393,5 @@
       link="Link6" />
     <axis
-      xyz="0 0 -1" />
+      xyz="0 0 1" />
     <limit
       lower="-6.28"

File: cra_description/urdf/cr7_robot.xacro (robot description, xacro)
@@ -101,5 +101,5 @@
       link="Link1" />
     <axis
-      xyz="0 0 -1" />
+      xyz="0 0 1" />
     <limit
       lower="-6.27"
@@ -333,5 +333,5 @@
       link="Link5" />
     <axis
-      xyz="0 0 -1" />
+      xyz="0 0 1" />
     <limit
       lower="-6.27"
@@ -391,5 +391,5 @@
       link="Link6" />
     <axis
-      xyz="0 0 -1" />
+      xyz="0 0 1" />
     <limit
       lower="-6.27"

File: cra_description/urdf/me6_robot.xacro (robot description, xacro)
@@ -208,9 +208,4 @@
         <limit lower="-6.27" upper="6.27" effort="300" velocity="300" />
     </joint>
-   <link name="world" />
-    <joint name="world_joint" type="fixed">
-        <parent link="world" />
-        <child link="dummy_link" />
-    </joint>
 <gazebo reference="base_link">
         <gravity>false</gravity>

File: cra_description/urdf/nova2_robot.xacro (robot description, xacro)
@@ -64,5 +64,5 @@
         <parent link="base_link" />
         <child link="Link1" />
-        <axis xyz="0 0 -1" />
+        <axis xyz="0 0 1" />
         <limit lower="-6.28" upper="6.28" effort="300" velocity="100" />
     </joint>
@@ -151,5 +151,5 @@
         <parent link="Link3" />
         <child link="Link4" />
-        <axis xyz="0 0 -1" />
+        <axis xyz="0 0 1" />
         <limit lower="-6.28" upper="6.28" effort="300" velocity="100" />
     </joint>
@@ -180,5 +180,5 @@
         <parent link="Link4" />
         <child link="Link5" />
-        <axis xyz="0 0 -1" />
+        <axis xyz="0 0 1" />
         <limit lower="-6.28" upper="6.28" effort="300" velocity="100" />
     </joint>

File: dobot_rviz/urdf/cr10af_robot.urdf (robot description, URDF)
Before this commit: robot cr10af_robot, 8 links, 7 joints
Links:
- removed link J1
- removed link J2
- removed link J3
- removed link J4
- removed link J5
- removed link J6
- added link Link1, mass 8.97; collision mesh filename=package://dobot_rviz/meshes/cr10af/J1.STL; visual mesh filename=package://dobot_rviz/meshes/cr10af/J1.STL
- added link Link2, mass 16.9; collision mesh filename=package://dobot_rviz/meshes/cr10af/J2.STL; visual mesh filename=package://dobot_rviz/meshes/cr10af/J2.STL
- added link Link3, mass 5.47; collision mesh filename=package://dobot_rviz/meshes/cr10af/J3.STL; visual mesh filename=package://dobot_rviz/meshes/cr10af/J3.STL
- added link Link4, mass 2.6; collision mesh filename=package://dobot_rviz/meshes/cr10af/J4.STL; visual mesh filename=package://dobot_rviz/meshes/cr10af/J4.STL
- added link Link5, mass 2.6; collision mesh filename=package://dobot_rviz/meshes/cr10af/J5.STL; visual mesh filename=package://dobot_rviz/meshes/cr10af/J5.STL
- added link Link6, mass 0.4; collision mesh filename=package://dobot_rviz/meshes/cr10af/J6.STL; visual mesh filename=package://dobot_rviz/meshes/cr10af/J6.STL
- added link tool0
Joints:
- added joint tool_joint: type fixed, parent Link6, child tool0, origin xyz=0 0 0 rpy=4.7124 0 3.14159
- joint joint1: child J1 -> Link1
- joint joint2: child J2 -> Link2; parent J1 -> Link1
- joint joint3: axis 0 1 0 -> 0 -1 0; child J3 -> Link3; parent J2 -> Link2
- joint joint4: child J4 -> Link4; parent J3 -> Link3
- joint joint5: child J5 -> Link5; parent J4 -> Link4
- joint joint6: child J6 -> Link6; parent J5 -> Link5

File: dobot_rviz/urdf/cr30h_robot.urdf (robot description, URDF)
Before this commit: robot cr30h_robot, 8 links, 7 joints
Joints:
- joint joint1: axis -1 0 0 -> 0 0 1; origin xyz=0 0 0.386 rpy=1.5708 1.5708 0 -> xyz=0 0 0.386 rpy=0 0 0
- joint joint6: axis 0 0 -1 -> 0 0 1

File: dobot_rviz/urdf/cr3_robot.urdf (robot description, URDF)
Before this commit: robot cr3_robot, 8 links, 7 joints
Joints:
- joint joint1: origin xyz=0 0 0.1348 rpy=0 0 -1.5708 -> xyz=0 0 0.1348 rpy=0 0 0
- joint joint4: axis 0 0 -1 -> 0 0 1
- joint joint5: axis 0 0 -1 -> 0 0 1
- joint joint6: axis 0 0 -1 -> 0 0 1

File: dobot_rviz/urdf/cr7_robot.urdf (robot description, URDF)
Before this commit: robot cr7_robot, 8 links, 7 joints
Joints:
- joint joint1: axis 0 0 -1 -> 0 0 1
- joint joint5: axis 0 0 -1 -> 0 0 1
- joint joint6: axis 0 0 -1 -> 0 0 1
