Commit message: V1.02

File: cra_description/urdf/cr10af_robot.xacro (robot description, xacro)
@@ -107,6 +107,6 @@
       lower="-6.2831"
       upper="6.2831"
-      effort="0"
-      velocity="0" />
+      effort="300"
+      velocity="3.14" />
   </joint>
   <link
@@ -165,6 +165,6 @@
       lower="-6.2831"
       upper="6.2831"
-      effort="0"
-      velocity="0" />
+      effort="300"
+      velocity="3.14" />
   </joint>
   <link
@@ -223,6 +223,6 @@
       lower="-2.7925"
       upper="2.7925"
-      effort="0"
-      velocity="0" />
+      effort="300"
+      velocity="3.14" />
   </joint>
   <link
@@ -281,6 +281,6 @@
       lower="-6.2831"
       upper="6.2831"
-      effort="0"
-      velocity="0" />
+      effort="300"
+      velocity="3.14" />
   </joint>
   <link
@@ -339,6 +339,6 @@
       lower="-6.2831"
       upper="6.2831"
-      effort="0"
-      velocity="0" />
+      effort="300"
+      velocity="3.14" />
   </joint>
   <link
@@ -397,6 +397,6 @@
       lower="-6.2831"
       upper="6.2831"
-      effort="0"
-      velocity="0" />
+      effort="300"
+      velocity="3.14" />
   </joint>
   <link name="tool0"/>
@@ -437,5 +437,5 @@
     <ros2_control name="GazeboSystem" type="system">
         <hardware>
-            <plugin>gazebo_ros2_control/GazeboSystem</plugin>
+            <plugin>gz_ros2_control/GazeboSimSystem</plugin>
         </hardware>
         <joint name="joint1">
@@ -501,5 +501,5 @@
     </ros2_control>
     <gazebo>
-        <plugin filename="libgazebo_ros2_control.so" name="gazebo_ros2_control">
+        <plugin filename="gz_ros2_control-system" name="gz_ros2_control::GazeboSimROS2ControlPlugin">
             <parameters>$(find cr10af_moveit)/config/ros2_controllers.yaml</parameters>
             <robot_param_node>robot_state_publisher</robot_param_node>

File: cra_description/urdf/cr20_robot.xacro (robot description, xacro)
@@ -108,6 +108,6 @@
       lower="-6.28"
       upper="6.28"
-      effort="0"
-      velocity="0" />
+      effort="300"
+      velocity="3.14" />
   </joint>
   <link
@@ -166,6 +166,6 @@
       lower="-6.28"
       upper="6.28"
-      effort="0"
-      velocity="0" />
+      effort="300"
+      velocity="3.14" />
   </joint>
   <link
@@ -224,6 +224,6 @@
       lower="-2.9"
       upper="2.9"
-      effort="0"
-      velocity="0" />
+      effort="300"
+      velocity="3.14" />
   </joint>
   <link
@@ -282,6 +282,6 @@
       lower="-6.28"
       upper="6.28"
-      effort="0"
-      velocity="0" />
+      effort="300"
+      velocity="3.14" />
   </joint>
   <link
@@ -340,6 +340,6 @@
       lower="-6.28"
       upper="6.28"
-      effort="0"
-      velocity="0" />
+      effort="300"
+      velocity="3.14" />
   </joint>
   <link
@@ -398,6 +398,6 @@
       lower="-6.28"
       upper="6.28"
-      effort="0"
-      velocity="0" />
+      effort="300"
+      velocity="3.14" />
   </joint>
     <gazebo reference="Link1">
@@ -428,5 +428,5 @@
     <ros2_control name="GazeboSystem" type="system">
         <hardware>
-            <plugin>gazebo_ros2_control/GazeboSystem</plugin>
+            <plugin>gz_ros2_control/GazeboSimSystem</plugin>
         </hardware>
         <joint name="joint1">
@@ -492,5 +492,5 @@
     </ros2_control>
     <gazebo>
-        <plugin filename="libgazebo_ros2_control.so" name="gazebo_ros2_control">
+        <plugin filename="gz_ros2_control-system" name="gz_ros2_control::GazeboSimROS2ControlPlugin">
             <parameters>$(find cr20_moveit)/config/ros2_controllers.yaml</parameters>
             <robot_param_node>robot_state_publisher</robot_param_node>

File: cra_description/urdf/cr30h_robot.xacro (robot description, xacro)
@@ -108,6 +108,6 @@
       lower="-6.28"
       upper="6.28"
-      effort="0"
-      velocity="0" />
+      effort="300"
+      velocity="3.14" />
   </joint>
   <link
@@ -166,6 +166,6 @@
       lower="-6.28"
       upper="6.28"
-      effort="0"
-      velocity="0" />
+      effort="300"
+      velocity="3.14" />
   </joint>
   <link
@@ -224,6 +224,6 @@
       lower="-2.79"
       upper="2.79"
-      effort="0"
-      velocity="0" />
+      effort="300"
+      velocity="3.14" />
   </joint>
   <link
@@ -282,6 +282,6 @@
       lower="-6.28"
       upper="6.28"
-      effort="0"
-      velocity="0" />
+      effort="300"
+      velocity="3.14" />
   </joint>
   <link
@@ -340,6 +340,6 @@
       lower="-6.28"
       upper="6.28"
-      effort="0"
-      velocity="0" />
+      effort="300"
+      velocity="3.14" />
   </joint>
   <link
@@ -398,6 +398,6 @@
       lower="-6.28"
       upper="6.28"
-      effort="0"
-      velocity="0" />
+      effort="300"
+      velocity="3.14" />
   </joint>
     <gazebo reference="Link1">
@@ -428,5 +428,5 @@
     <ros2_control name="GazeboSystem" type="system">
         <hardware>
-            <plugin>gazebo_ros2_control/GazeboSystem</plugin>
+            <plugin>gz_ros2_control/GazeboSimSystem</plugin>
         </hardware>
         <joint name="joint1">
@@ -492,5 +492,5 @@
     </ros2_control>
     <gazebo>
-        <plugin filename="libgazebo_ros2_control.so" name="gazebo_ros2_control">
+        <plugin filename="gz_ros2_control-system" name="gz_ros2_control::GazeboSimROS2ControlPlugin">
             <parameters>$(find cr30h_moveit)/config/ros2_controllers.yaml</parameters>
             <robot_param_node>robot_state_publisher</robot_param_node>

File: cra_description/urdf/cr3_robot.xacro (robot description, xacro)
@@ -107,6 +107,6 @@
       lower="-6.28"
       upper="6.28"
-      effort="0"
-      velocity="0" />
+      effort="300"
+      velocity="3.14" />
   </joint>
   <link
@@ -165,6 +165,6 @@
       lower="-6.28"
       upper="6.28"
-      effort="0"
-      velocity="0" />
+      effort="300"
+      velocity="3.14" />
   </joint>
   <link
@@ -223,6 +223,6 @@
       lower="-2.7039"
       upper="2.7039"
-      effort="0"
-      velocity="0" />
+      effort="300"
+      velocity="3.14" />
   </joint>
   <link
@@ -281,6 +281,6 @@
       lower="-6.28"
       upper="6.28"
-      effort="0"
-      velocity="0" />
+      effort="300"
+      velocity="3.14" />
   </joint>
   <link
@@ -339,6 +339,6 @@
       lower="-6.28"
       upper="6.28"
-      effort="0"
-      velocity="0" />
+      effort="300"
+      velocity="3.14" />
   </joint>
   <link
@@ -397,6 +397,6 @@
       lower="-6.28"
       upper="6.28"
-      effort="0"
-      velocity="0" />
+      effort="300"
+      velocity="3.14" />
   </joint>
     <gazebo reference="base_link">
@@ -431,5 +431,5 @@
     <ros2_control name="GazeboSystem" type="system">
         <hardware>
-            <plugin>gazebo_ros2_control/GazeboSystem</plugin>
+            <plugin>gz_ros2_control/GazeboSimSystem</plugin>
         </hardware>
         <joint name="joint1">
@@ -495,5 +495,5 @@
     </ros2_control>
     <gazebo>
-        <plugin filename="libgazebo_ros2_control.so" name="gazebo_ros2_control">
+        <plugin filename="gz_ros2_control-system" name="gz_ros2_control::GazeboSimROS2ControlPlugin">
             <parameters>$(find cr3_moveit)/config/ros2_controllers.yaml</parameters>
             <robot_param_node>robot_state_publisher</robot_param_node>

File: cra_description/urdf/cr5_robot.xacro (robot description, xacro)
@@ -107,6 +107,6 @@
       lower="-6.28"
       upper="6.28"
-      effort="0"
-      velocity="0" />
+      effort="300"
+      velocity="3.14" />
   </joint>
   <link
@@ -165,6 +165,6 @@
       lower="-6.28"
       upper="6.28"
-      effort="0"
-      velocity="0" />
+      effort="300"
+      velocity="3.14" />
   </joint>
   <link
@@ -223,6 +223,6 @@
       lower="-2.792"
       upper="2.792"
-      effort="0"
-      velocity="0" />
+      effort="300"
+      velocity="3.14" />
   </joint>
   <link
@@ -281,6 +281,6 @@
       lower="-6.28"
       upper="6.28"
-      effort="0"
-      velocity="0" />
+      effort="300"
+      velocity="3.14" />
   </joint>
   <link
@@ -339,6 +339,6 @@
       lower="-6.28"
       upper="6.28"
-      effort="0"
-      velocity="0" />
+      effort="300"
+      velocity="3.14" />
   </joint>
   <link
@@ -397,6 +397,6 @@
       lower="-6.28"
       upper="6.28"
-      effort="0"
-      velocity="0" />
+      effort="300"
+      velocity="3.14" />
   </joint>
     <gazebo reference="base_link">
@@ -431,5 +431,5 @@
     <ros2_control name="GazeboSystem" type="system">
         <hardware>
-            <plugin>gazebo_ros2_control/GazeboSystem</plugin>
+            <plugin>gz_ros2_control/GazeboSimSystem</plugin>
         </hardware>
         <joint name="joint1">
@@ -495,5 +495,5 @@
     </ros2_control>
     <gazebo>
-        <plugin filename="libgazebo_ros2_control.so" name="gazebo_ros2_control">
+        <plugin filename="gz_ros2_control-system" name="gz_ros2_control::GazeboSimROS2ControlPlugin">
             <parameters> $(find cr5_moveit)/config/ros2_controllers.yaml</parameters>
             <robot_param_node>robot_state_publisher</robot_param_node>

File: cra_description/urdf/nova5_robot.xacro (robot description, xacro)
@@ -111,6 +111,6 @@
       lower="-6.28"
       upper="6.28"
-      effort="0"
-      velocity="0" />
+      effort="300"
+      velocity="3.14" />
   </joint>
   <link
@@ -169,6 +169,6 @@
       lower="-3.14"
       upper="3.14"
-      effort="0"
-      velocity="0" />
+      effort="300"
+      velocity="3.14" />
   </joint>
   <link
@@ -227,6 +227,6 @@
       lower="-2.79"
       upper="2.79"
-      effort="0"
-      velocity="0" />
+      effort="300"
+      velocity="3.14" />
   </joint>
   <link
@@ -285,6 +285,6 @@
       lower="-6.28"
       upper="6.28"
-      effort="0"
-      velocity="0" />
+      effort="300"
+      velocity="3.14" />
   </joint>
   <link
@@ -343,6 +343,6 @@
       lower="-6.28"
       upper="6.28"
-      effort="0"
-      velocity="0" />
+      effort="300"
+      velocity="3.14" />
   </joint>
   <link
@@ -401,6 +401,6 @@
       lower="-6.28"
       upper="6.28"
-      effort="0"
-      velocity="0" />
+      effort="300"
+      velocity="3.14" />
   </joint>
    <gazebo reference="base_link">
@@ -435,5 +435,5 @@
     <ros2_control name="GazeboSystem" type="system">
         <hardware>
-            <plugin>gazebo_ros2_control/GazeboSystem</plugin>
+            <plugin>gz_ros2_control/GazeboSimSystem</plugin>
         </hardware>
         <joint name="joint1">
@@ -499,5 +499,5 @@
     </ros2_control>
     <gazebo>
-        <plugin filename="libgazebo_ros2_control.so" name="gazebo_ros2_control">
+        <plugin filename="gz_ros2_control-system" name="gz_ros2_control::GazeboSimROS2ControlPlugin">
             <parameters> $(find nova5_moveit)/config/ros2_controllers.yaml</parameters>
             <robot_param_node>robot_state_publisher</robot_param_node>

File: dobot_rviz/urdf/cr10_robot.urdf (robot description, URDF)
Before this commit: robot cr10_robot, 8 links, 7 joints
Links:
- removed link dummy_link
Joints:
- removed joint dummy_joint
- joint joint1: limit lower=-6.27 upper=6.27 effort=0 velocity=0 -> lower=-6.27 upper=6.27 effort=0 velocity=0.5236
- joint joint2: limit lower=-6.27 upper=6.27 effort=0 velocity=0 -> lower=-6.27 upper=6.27 effort=0 velocity=0.5236
- joint joint3: limit lower=-2.861 upper=2.861 effort=0 velocity=0 -> lower=-2.861 upper=2.861 effort=0 velocity=0.5236
- joint joint4: limit lower=-6.27 upper=6.27 effort=0 velocity=0 -> lower=-6.27 upper=6.27 effort=0 velocity=0.5236
- joint joint5: limit lower=-6.27 upper=6.27 effort=0 velocity=0 -> lower=-6.27 upper=6.27 effort=0 velocity=0.5236
- joint joint6: limit lower=-6.27 upper=6.27 effort=0 velocity=0 -> lower=-6.27 upper=6.27 effort=0 velocity=0.5236

File: dobot_rviz/urdf/cr10af_robot.urdf (robot description, URDF)
Before this commit: robot cr10af_robot, 9 links, 8 joints
Links:
- removed link dummy_link
Joints:
- removed joint dummy_joint
- joint joint1: limit lower=-6.2831 upper=6.2831 effort=0 velocity=0 -> lower=-6.2831 upper=6.2831 effort=0 velocity=0.5236
- joint joint2: limit lower=-6.2831 upper=6.2831 effort=0 velocity=0 -> lower=-6.2831 upper=6.2831 effort=0 velocity=0.5236
- joint joint3: limit lower=-2.7925 upper=2.7925 effort=0 velocity=0 -> lower=-2.7925 upper=2.7925 effort=0 velocity=0.5236
- joint joint4: limit lower=-6.2831 upper=6.2831 effort=0 velocity=0 -> lower=-6.2831 upper=6.2831 effort=0 velocity=0.5236
- joint joint5: limit lower=-6.2831 upper=6.2831 effort=0 velocity=0 -> lower=-6.2831 upper=6.2831 effort=0 velocity=0.5236
- joint joint6: limit lower=-6.2831 upper=6.2831 effort=0 velocity=0 -> lower=-6.2831 upper=6.2831 effort=0 velocity=0.5236

File: dobot_rviz/urdf/cr12_robot.urdf (robot description, URDF)
Before this commit: robot cr12_robot, 8 links, 7 joints
Links:
- removed link dummy_link
Joints:
- removed joint dummy_joint
- joint joint1: limit lower=-6.27 upper=6.27 effort=0 velocity=0 -> lower=-6.27 upper=6.27 effort=0 velocity=0.5236
- joint joint2: limit lower=-6.27 upper=6.27 effort=0 velocity=0 -> lower=-6.27 upper=6.27 effort=0 velocity=0.5236
- joint joint3: limit lower=-2.79 upper=2.79 effort=0 velocity=0 -> lower=-2.79 upper=2.79 effort=0 velocity=0.5236
- joint joint4: limit lower=-6.27 upper=6.27 effort=0 velocity=0 -> lower=-6.27 upper=6.27 effort=0 velocity=0.5236
- joint joint5: limit lower=-6.27 upper=6.27 effort=0 velocity=0 -> lower=-6.27 upper=6.27 effort=0 velocity=0.5236
- joint joint6: limit lower=-6.27 upper=6.27 effort=0 velocity=0 -> lower=-6.27 upper=6.27 effort=0 velocity=0.5236

File: dobot_rviz/urdf/cr16_robot.urdf (robot description, URDF)
Before this commit: robot cr16_robot, 8 links, 7 joints
Links:
- removed link dummy_link
Joints:
- removed joint dummy_joint
- joint joint1: limit lower=-6.27 upper=6.27 effort=0 velocity=0 -> lower=-6.27 upper=6.27 effort=0 velocity=0.5236
- joint joint2: limit lower=-6.27 upper=6.27 effort=0 velocity=0 -> lower=-6.27 upper=6.27 effort=0 velocity=0.5236
- joint joint3: limit lower=-2.86 upper=2.86 effort=0 velocity=0 -> lower=-2.86 upper=2.86 effort=0 velocity=0.5236
- joint joint4: limit lower=-6.27 upper=6.27 effort=0 velocity=0 -> lower=-6.27 upper=6.27 effort=0 velocity=0.5236
- joint joint5: limit lower=-6.27 upper=6.27 effort=0 velocity=0 -> lower=-6.27 upper=6.27 effort=0 velocity=0.5236
- joint joint6: limit lower=-6.27 upper=6.27 effort=0 velocity=0 -> lower=-6.27 upper=6.27 effort=0 velocity=0.5236

File: dobot_rviz/urdf/cr20_robot.urdf (robot description, URDF)
Before this commit: robot cr20_robot, 8 links, 7 joints
Links:
- removed link dummy_link
Joints:
- removed joint dummy_joint
- joint joint1: limit lower=-6.28 upper=6.28 effort=0 velocity=0 -> lower=-6.28 upper=6.28 effort=0 velocity=0.5236
- joint joint2: limit lower=-6.28 upper=6.28 effort=0 velocity=0 -> lower=-6.28 upper=6.28 effort=0 velocity=0.5236
- joint joint3: limit lower=-2.9 upper=2.9 effort=0 velocity=0 -> lower=-2.9 upper=2.9 effort=0 velocity=0.5236
- joint joint4: limit lower=-6.28 upper=6.28 effort=0 velocity=0 -> lower=-6.28 upper=6.28 effort=0 velocity=0.5236
- joint joint5: limit lower=-6.28 upper=6.28 effort=0 velocity=0 -> lower=-6.28 upper=6.28 effort=0 velocity=0.5236
- joint joint6: limit lower=-6.28 upper=6.28 effort=0 velocity=0 -> lower=-6.28 upper=6.28 effort=0 velocity=0.5236

File: dobot_rviz/urdf/cr30h_robot.urdf (robot description, URDF)
Before this commit: robot cr30h_robot, 8 links, 7 joints
Links:
- removed link dummy_link
Joints:
- removed joint dummy_joint
- joint joint1: limit lower=-6.28 upper=6.28 effort=0 velocity=0 -> lower=-6.28 upper=6.28 effort=0 velocity=0.5236
- joint joint2: limit lower=-6.28 upper=6.28 effort=0 velocity=0 -> lower=-6.28 upper=6.28 effort=0 velocity=0.5236
- joint joint3: limit lower=-2.79 upper=2.79 effort=0 velocity=0 -> lower=-2.79 upper=2.79 effort=0 velocity=0.5236
- joint joint4: limit lower=-6.28 upper=6.28 effort=0 velocity=0 -> lower=-6.28 upper=6.28 effort=0 velocity=0.5236
- joint joint5: limit lower=-6.28 upper=6.28 effort=0 velocity=0 -> lower=-6.28 upper=6.28 effort=0 velocity=0.5236
- joint joint6: limit lower=-6.28 upper=6.28 effort=0 velocity=0 -> lower=-6.28 upper=6.28 effort=0 velocity=0.5236

File: dobot_rviz/urdf/cr3_robot.urdf (robot description, URDF)
Before this commit: robot cr3_robot, 8 links, 7 joints
Links:
- removed link dummy_link
Joints:
- removed joint dummy_joint
- joint joint1: limit lower=-6.28 upper=6.28 effort=0 velocity=0 -> lower=-6.28 upper=6.28 effort=0 velocity=0.5236
- joint joint2: limit lower=-6.28 upper=6.28 effort=0 velocity=0 -> lower=-6.28 upper=6.28 effort=0 velocity=0.5236
- joint joint3: limit lower=-2.7039 upper=2.7039 effort=0 velocity=0 -> lower=-2.7039 upper=2.7039 effort=0 velocity=0.5236
- joint joint4: limit lower=-6.28 upper=6.28 effort=0 velocity=0 -> lower=-6.28 upper=6.28 effort=0 velocity=0.5236
- joint joint5: limit lower=-6.28 upper=6.28 effort=0 velocity=0 -> lower=-6.28 upper=6.28 effort=0 velocity=0.5236
- joint joint6: limit lower=-6.28 upper=6.28 effort=0 velocity=0 -> lower=-6.28 upper=6.28 effort=0 velocity=0.5236

File: dobot_rviz/urdf/cr5_robot.urdf (robot description, URDF)
Before this commit: robot cr5_robot, 8 links, 7 joints
Links:
- removed link dummy_link
Joints:
- removed joint dummy_joint
- joint joint1: limit lower=-6.28 upper=6.28 effort=0 velocity=0 -> lower=-6.28 upper=6.28 effort=0 velocity=0.5236
- joint joint2: limit lower=-6.28 upper=6.28 effort=0 velocity=0 -> lower=-6.28 upper=6.28 effort=0 velocity=0.5236
- joint joint3: limit lower=-2.792 upper=2.792 effort=0 velocity=0 -> lower=-2.792 upper=2.792 effort=0 velocity=0.5236
- joint joint4: limit lower=-6.28 upper=6.28 effort=0 velocity=0 -> lower=-6.28 upper=6.28 effort=0 velocity=0.5236
- joint joint5: limit lower=-6.28 upper=6.28 effort=0 velocity=0 -> lower=-6.28 upper=6.28 effort=0 velocity=0.5236
- joint joint6: limit lower=-6.28 upper=6.28 effort=0 velocity=0 -> lower=-6.28 upper=6.28 effort=0 velocity=0.5236

File: dobot_rviz/urdf/cr7_robot.urdf (robot description, URDF)
Before this commit: robot cr7_robot, 8 links, 7 joints
Links:
- removed link dummy_link
Joints:
- removed joint dummy_joint
- joint joint1: limit lower=-6.27 upper=6.27 effort=0 velocity=0 -> lower=-6.27 upper=6.27 effort=0 velocity=0.5236
- joint joint2: limit lower=-6.27 upper=6.27 effort=0 velocity=0 -> lower=-6.27 upper=6.27 effort=0 velocity=0.5236
- joint joint3: limit lower=-2.79 upper=2.79 effort=0 velocity=0 -> lower=-2.79 upper=2.79 effort=0 velocity=0.5236
- joint joint4: limit lower=-6.27 upper=6.27 effort=0 velocity=0 -> lower=-6.27 upper=6.27 effort=0 velocity=0.5236
- joint joint5: limit lower=-6.27 upper=6.27 effort=0 velocity=0 -> lower=-6.27 upper=6.27 effort=0 velocity=0.5236
- joint joint6: limit lower=-6.27 upper=6.27 effort=0 velocity=0 -> lower=-6.27 upper=6.27 effort=0 velocity=0.5236

File: dobot_rviz/urdf/me6_robot.urdf (robot description, URDF)
Before this commit: robot me6_robot, 8 links, 7 joints
Links:
- removed link dummy_link
Joints:
- removed joint dummy_joint
- joint joint1: limit lower=-6.27 upper=6.27 effort=0 velocity=0 -> lower=-6.27 upper=6.27 effort=0 velocity=0.5236
- joint joint2: limit lower=-2.356 upper=2.356 effort=0 velocity=0 -> lower=-2.356 upper=2.356 effort=0 velocity=0.5236
- joint joint3: limit lower=-2.6878 upper=2.6878 effort=0 velocity=0 -> lower=-2.6878 upper=2.6878 effort=0 velocity=0.5236
- joint joint4: limit lower=-2.7925 upper=2.7925 effort=0 velocity=0 -> lower=-2.7925 upper=2.7925 effort=0 velocity=0.5236
- joint joint5: limit lower=-3.0194 upper=3.0194 effort=0 velocity=0 -> lower=-3.0194 upper=3.0194 effort=0 velocity=0.5236
- joint joint6: limit lower=-6.27 upper=6.27 effort=0 velocity=0 -> lower=-6.27 upper=6.27 effort=0 velocity=0.5236

File: dobot_rviz/urdf/nova2_robot.urdf (robot description, URDF)
Before this commit: robot nova2_robot, 8 links, 7 joints
Links:
- removed link dummy_link
Joints:
- removed joint dummy_joint
- joint joint1: limit lower=-6.28 upper=6.28 effort=0 velocity=0 -> lower=-6.28 upper=6.28 effort=0 velocity=0.5236
- joint joint2: limit lower=-3.14 upper=3.14 effort=0 velocity=0 -> lower=-3.14 upper=3.14 effort=0 velocity=0.5236
- joint joint3: limit lower=-2.79 upper=2.79 effort=0 velocity=0 -> lower=-2.79 upper=2.79 effort=0 velocity=0.5236
- joint joint4: limit lower=-6.28 upper=6.28 effort=0 velocity=0 -> lower=-6.28 upper=6.28 effort=0 velocity=0.5236
- joint joint5: limit lower=-6.28 upper=6.28 effort=0 velocity=0 -> lower=-6.28 upper=6.28 effort=0 velocity=0.5236
- joint joint6: limit lower=-6.28 upper=6.28 effort=0 velocity=0 -> lower=-6.28 upper=6.28 effort=0 velocity=0.5236

File: dobot_rviz/urdf/nova5_robot.urdf (robot description, URDF)
Before this commit: robot nova5_robot, 8 links, 7 joints
Links:
- removed link dummy_link
Joints:
- removed joint dummy_joint
- joint joint1: limit lower=-6.28 upper=6.28 effort=0 velocity=0 -> lower=-6.28 upper=6.28 effort=0 velocity=0.5236
- joint joint2: limit lower=-3.14 upper=3.14 effort=0 velocity=0 -> lower=-3.14 upper=3.14 effort=0 velocity=0.5236
- joint joint3: limit lower=-2.79 upper=2.79 effort=0 velocity=0 -> lower=-2.79 upper=2.79 effort=0 velocity=0.5236
- joint joint4: limit lower=-6.28 upper=6.28 effort=0 velocity=0 -> lower=-6.28 upper=6.28 effort=0 velocity=0.5236
- joint joint5: limit lower=-6.28 upper=6.28 effort=0 velocity=0 -> lower=-6.28 upper=6.28 effort=0 velocity=0.5236
- joint joint6: limit lower=-6.28 upper=6.28 effort=0 velocity=0 -> lower=-6.28 upper=6.28 effort=0 velocity=0.5236
