Commit message: fix: Fixed multi-robot configuration issues and improved joint status forwarding Fix the rviz target coordinate system of all moveit configurations from dummy_link to base_link 2. Reconstruct the dummy joint and world joint layout of the robot description package 3. Remove the redundant joint_states nodes in dobot_moveit and add the joint state forwarding script 4. Complete all dependencies and correct the default values of the environment variables in the launch file 5. Adjust the controller parameters and urdf joint limit parameters 6. Correct the joint axis direction and initial posture of the cr30h robot

File: cr10_moveit/config/cr10_robot.ros2_control.xacro (robot description, xacro)
@@ -2,5 +2,5 @@
 <robot xmlns:xacro="http://www.ros.org/wiki/xacro">
     <xacro:macro name="cr10_robot_ros2_control" params="name initial_positions_file">
-        <xacro:property name="initial_positions" value="${load_yaml(initial_positions_file)['initial_positions']}"/>
+        <xacro:property name="initial_positions" value="${xacro.load_yaml(initial_positions_file)['initial_positions']}"/>
         <ros2_control name="${name}" type="system">
             <hardware>

File: cr10af_moveit/config/cr10af_robot.ros2_control.xacro (robot description, xacro)
@@ -2,5 +2,5 @@
 <robot xmlns:xacro="http://www.ros.org/wiki/xacro">
     <xacro:macro name="cr10af_robot_ros2_control" params="name initial_positions_file">
-        <xacro:property name="initial_positions" value="${load_yaml(initial_positions_file)['initial_positions']}"/>
+        <xacro:property name="initial_positions" value="${xacro.load_yaml(initial_positions_file)['initial_positions']}"/>
         <ros2_control name="${name}" type="system">
             <hardware>

File: cr12_moveit/config/cr12_robot.ros2_control.xacro (robot description, xacro)
@@ -2,5 +2,5 @@
 <robot xmlns:xacro="http://www.ros.org/wiki/xacro">
     <xacro:macro name="cr12_robot_ros2_control" params="name initial_positions_file">
-        <xacro:property name="initial_positions" value="${load_yaml(initial_positions_file)['initial_positions']}"/>
+        <xacro:property name="initial_positions" value="${xacro.load_yaml(initial_positions_file)['initial_positions']}"/>
         <ros2_control name="${name}" type="system">
             <hardware>

File: cr16_moveit/config/cr16_robot.ros2_control.xacro (robot description, xacro)
@@ -2,5 +2,5 @@
 <robot xmlns:xacro="http://www.ros.org/wiki/xacro">
     <xacro:macro name="cr16_robot_ros2_control" params="name initial_positions_file">
-        <xacro:property name="initial_positions" value="${load_yaml(initial_positions_file)['initial_positions']}"/>
+        <xacro:property name="initial_positions" value="${xacro.load_yaml(initial_positions_file)['initial_positions']}"/>
         <ros2_control name="${name}" type="system">
             <hardware>

File: cr20_moveit/config/cr20_robot.ros2_control.xacro (robot description, xacro)
@@ -2,5 +2,5 @@
 <robot xmlns:xacro="http://www.ros.org/wiki/xacro">
     <xacro:macro name="cr20_robot_ros2_control" params="name initial_positions_file">
-        <xacro:property name="initial_positions" value="${load_yaml(initial_positions_file)['initial_positions']}"/>
+        <xacro:property name="initial_positions" value="${xacro.load_yaml(initial_positions_file)['initial_positions']}"/>
         <ros2_control name="${name}" type="system">
             <hardware>

File: cr30h_moveit/config/cr30h_robot.ros2_control.xacro (robot description, xacro)
@@ -2,5 +2,5 @@
 <robot xmlns:xacro="http://www.ros.org/wiki/xacro">
     <xacro:macro name="cr30h_robot_ros2_control" params="name initial_positions_file">
-        <xacro:property name="initial_positions" value="${load_yaml(initial_positions_file)['initial_positions']}"/>
+        <xacro:property name="initial_positions" value="${xacro.load_yaml(initial_positions_file)['initial_positions']}"/>
         <ros2_control name="${name}" type="system">
             <hardware>

File: cr3_moveit/config/cr3_robot.ros2_control.xacro (robot description, xacro)
@@ -2,5 +2,5 @@
 <robot xmlns:xacro="http://www.ros.org/wiki/xacro">
     <xacro:macro name="cr3_robot_ros2_control" params="name initial_positions_file">
-        <xacro:property name="initial_positions" value="${load_yaml(initial_positions_file)['initial_positions']}"/>
+        <xacro:property name="initial_positions" value="${xacro.load_yaml(initial_positions_file)['initial_positions']}"/>
         <ros2_control name="${name}" type="system">
             <hardware>

File: cr5_moveit/config/cr5_robot.ros2_control.xacro (robot description, xacro)
@@ -2,5 +2,5 @@
 <robot xmlns:xacro="http://www.ros.org/wiki/xacro">
     <xacro:macro name="cr5_robot_ros2_control" params="name initial_positions_file">
-        <xacro:property name="initial_positions" value="${load_yaml(initial_positions_file)['initial_positions']}"/>
+        <xacro:property name="initial_positions" value="${xacro.load_yaml(initial_positions_file)['initial_positions']}"/>
         <ros2_control name="${name}" type="system">
             <hardware>

File: cr7_moveit/config/cr7_robot.ros2_control.xacro (robot description, xacro)
@@ -2,5 +2,5 @@
 <robot xmlns:xacro="http://www.ros.org/wiki/xacro">
     <xacro:macro name="cr7_robot_ros2_control" params="name initial_positions_file">
-        <xacro:property name="initial_positions" value="${load_yaml(initial_positions_file)['initial_positions']}"/>
+        <xacro:property name="initial_positions" value="${xacro.load_yaml(initial_positions_file)['initial_positions']}"/>
         <ros2_control name="${name}" type="system">
             <hardware>

File: cra_description/urdf/cr10_robot.xacro (robot description, xacro)
@@ -1,6 +1,5 @@
 <?xml version="1.0"?>
 <robot name="cr10_robot" xmlns:xacro="http://ros.org/wiki/xacro">
-  <link name="dummy_link"/>
-  <link name="base_link">
+  <link name="dummy_link" /><link name="base_link">
     <inertial>
       <origin
@@ -40,4 +39,8 @@
     </collision>
   </link>
+  <joint name="dummy_joint" type="fixed">
+      <parent link="dummy_link" />
+      <child  link="base_link" />
+    </joint>
   <link  name="world"/>
 <joint name="world_joint" type="fixed">
@@ -45,10 +48,5 @@
     <parent link="world" />
     <child  link="dummy_link" />
-  </joint>
-  <joint name="dummy_joint" type="fixed">
-    <parent link="dummy_link" />
-    <child  link="base_link" />
-  </joint>
-  <link
+  </joint><link
     name="Link1">
     <inertial>

File: cra_description/urdf/cr10af_robot.xacro (robot description, xacro)
@@ -1,6 +1,5 @@
 <?xml version="1.0"?>
 <robot name="cr10af_robot" xmlns:xacro="http://ros.org/wiki/xacro">
-  <link name="dummy_link"/>
-  <link
+  <link name="dummy_link" /><link
     name="base_link">
     <inertial>
@@ -42,4 +41,8 @@
     </collision>
   </link>
+  <joint name="dummy_joint" type="fixed">
+      <parent link="dummy_link" />
+      <child  link="base_link" />
+    </joint>
     <link  name="world"/>
 <joint name="world_joint" type="fixed">
@@ -47,10 +50,5 @@
     <parent link="world" />
     <child  link="dummy_link" />
-  </joint>
-  <joint name="dummy_joint" type="fixed">
-      <parent link="dummy_link" />
-      <child  link="base_link" />
-    </joint>
-  <link
+  </joint><link
     name="Link1">
     <inertial>

File: cra_description/urdf/cr12_robot.xacro (robot description, xacro)
@@ -2,6 +2,5 @@
 <robot
   name="cr12_robot"  xmlns:xacro="http://ros.org/wiki/xacro">
-  <link name="dummy_link"/>
-  <link name="base_link">
+  <link name="dummy_link" /><link name="base_link">
     <inertial>
       <origin
@@ -40,4 +39,8 @@
     </collision>
   </link>
+  <joint name="dummy_joint" type="fixed">
+      <parent link="dummy_link" />
+      <child  link="base_link" />
+    </joint>
   <link  name="world"/>
 <joint name="world_joint" type="fixed">
@@ -45,10 +48,5 @@
     <parent link="world" />
     <child  link="dummy_link" />
-  </joint>
-  <joint name="dummy_joint" type="fixed">
-      <parent link="dummy_link" />
-      <child  link="base_link" />
-  </joint>
-  <link
+  </joint><link
     name="Link1">
     <inertial>

File: cra_description/urdf/cr16_robot.xacro (robot description, xacro)
@@ -1,6 +1,5 @@
 <?xml version="1.0"?>
 <robot name="cr16_robot" xmlns:xacro="http://ros.org/wiki/xacro">
-  <link name="dummy_link"/>
-  <link
+  <link name="dummy_link" /><link
     name="base_link">
     <inertial>
@@ -42,4 +41,8 @@
     </collision>
   </link>
+  <joint name="dummy_joint" type="fixed">
+      <parent link="dummy_link" />
+      <child  link="base_link" />
+    </joint>
   <link  name="world"/>
 <joint name="world_joint" type="fixed">
@@ -47,10 +50,5 @@
     <parent link="world" />
     <child  link="dummy_link" />
-  </joint>
-  <joint name="dummy_joint" type="fixed">
-    <parent link="dummy_link" />
-    <child  link="base_link" />
-  </joint>
-  <link
+  </joint><link
     name="Link1">
     <inertial>

File: cra_description/urdf/cr20_robot.xacro (robot description, xacro)
@@ -2,6 +2,5 @@
 <robot
   name="cr20_robot" xmlns:xacro="http://ros.org/wiki/xacro">
-  <link name="dummy_link"/>
-  <link
+  <link name="dummy_link" /><link
     name="base_link">
     <inertial>
@@ -43,4 +42,8 @@
     </collision>
   </link>
+  <joint name="dummy_joint" type="fixed">
+      <parent link="dummy_link" />
+      <child  link="base_link" />
+    </joint>
     <link  name="world"/>
   <joint name="world_joint" type="fixed">
@@ -48,10 +51,5 @@
     <parent link="world" />
     <child  link="dummy_link" />
-  </joint>
-  <joint name="dummy_joint" type="fixed">
-    <parent link="dummy_link" />
-    <child  link="base_link" />
-  </joint>
-  <link
+  </joint><link
     name="Link1">
     <inertial>

File: cra_description/urdf/cr30h_robot.xacro (robot description, xacro)
@@ -2,6 +2,5 @@
 <robot
   name="cr30h_robot" xmlns:xacro="http://ros.org/wiki/xacro">
-  <link name="dummy_link"/>
-  <link
+  <link name="dummy_link" /><link
     name="base_link">
     <inertial>
@@ -43,4 +42,8 @@
     </collision>
   </link>
+  <joint name="dummy_joint" type="fixed">
+      <parent link="dummy_link" />
+      <child  link="base_link" />
+    </joint>
   <link  name="world"/>
   <joint name="world_joint" type="fixed">
@@ -48,10 +51,5 @@
     <parent link="world" />
     <child  link="dummy_link" />
-  </joint>
-  <joint name="dummy_joint" type="fixed">
-      <parent link="dummy_link" />
-      <child  link="base_link" />
-    </joint>
-  <link
+  </joint><link
     name="Link1">
     <inertial>
@@ -98,5 +96,5 @@
     <origin
       xyz="0 0 0.386"
-      rpy="0 0 0" />
+      rpy="1.5708 1.5708 0" />
     <parent
       link="base_link" />
@@ -104,5 +102,5 @@
       link="Link1" />
     <axis
-      xyz="0 0 1" />
+      xyz="-1 0 0" />
     <limit
       lower="-6.28"
@@ -394,5 +392,5 @@
       link="Link6" />
     <axis
-      xyz="0 0 1" />
+      xyz="0 0 -1" />
     <limit
       lower="-6.28"

File: cra_description/urdf/cr3_robot.xacro (robot description, xacro)
@@ -1,6 +1,5 @@
 <?xml version="1.0"?>
 <robot name="cr3_robot" xmlns:xacro="http://ros.org/wiki/xacro">
-  <link name="dummy_link" />
-  <link
+  <link name="dummy_link" /><link
     name="base_link">
     <inertial>
@@ -42,4 +41,8 @@
     </collision>
   </link>
+  <joint name="dummy_joint" type="fixed">
+      <parent link="dummy_link" />
+      <child  link="base_link" />
+    </joint>
   <link  name="world"/>
   <joint name="world_joint" type="fixed">
@@ -47,10 +50,5 @@
     <parent link="world" />
     <child  link="dummy_link" />
-  </joint>
-  <joint name="dummy_joint" type="fixed">
-      <parent link="dummy_link" />
-      <child  link="base_link" />
-    </joint>
-  <link
+  </joint><link
     name="Link1">
     <inertial>

File: cra_description/urdf/cr5_robot.xacro (robot description, xacro)
@@ -1,6 +1,5 @@
 <?xml version="1.0"?>
 <robot name="cr5_robot" xmlns:xacro="http://ros.org/wiki/xacro">
-  <link name="dummy_link" />
-  <link
+  <link name="dummy_link" /><link
     name="base_link">
     <inertial>
@@ -42,4 +41,8 @@
     </collision>
   </link>
+  <joint name="dummy_joint" type="fixed">
+      <parent link="dummy_link" />
+      <child  link="base_link" />
+    </joint>
   <link  name="world"/>
   <joint name="world_joint" type="fixed">
@@ -47,10 +50,5 @@
     <parent link="world" />
     <child  link="dummy_link" />
-  </joint>
-  <joint name="dummy_joint" type="fixed">
-      <parent link="dummy_link" />
-      <child  link="base_link" />
-    </joint>
-  <link
+  </joint><link
     name="Link1">
     <inertial>

File: cra_description/urdf/cr7_robot.xacro (robot description, xacro)
@@ -1,6 +1,5 @@
 <?xml version="1.0"?>
 <robot name="cr7_robot"  xmlns:xacro="http://ros.org/wiki/xacro">
-    <link name="dummy_link" />
-  <link name="base_link">
+  <link name="dummy_link" /><link name="base_link">
     <inertial>
       <origin
@@ -40,4 +39,8 @@
     </collision>
   </link>
+  <joint name="dummy_joint" type="fixed">
+      <parent link="dummy_link" />
+      <child  link="base_link" />
+    </joint>
 <link  name="world"/>
 <joint name="world_joint" type="fixed">
@@ -45,10 +48,5 @@
     <parent link="world" />
     <child  link="dummy_link" />
-  </joint>
-  <joint name="dummy_joint" type="fixed">
-    <parent link="dummy_link" />
-    <child  link="base_link" />
-  </joint>
-  <link
+  </joint><link
     name="Link1">
     <inertial>

File: cra_description/urdf/me6_robot.xacro (robot description, xacro)
@@ -1,6 +1,5 @@
 <?xml version="1.0" ?>
 <robot name="me6_robot" xmlns:xacro="http://www.ros.org/wiki/xacro">
-    <link name="dummy_link" />
-    <link name="base_link">
+  <link name="dummy_link" /><link name="base_link">
 <inertial>
             <origin xyz="-0.0240568795993814 0.00375533156407527 0.0319345452713943" rpy="0 0 0" />
@@ -24,4 +23,8 @@
         </collision>
     </link>
+  <joint name="dummy_joint" type="fixed">
+      <parent link="dummy_link" />
+      <child  link="base_link" />
+    </joint>
     <link  name="world"/>
   <joint name="world_joint" type="fixed">
@@ -29,10 +32,5 @@
     <parent link="world" />
     <child  link="dummy_link" />
-  </joint>
-    <joint name="dummy_joint" type="fixed">
-        <parent link="dummy_link" />
-        <child link="base_link" />
-    </joint>
-    <link name="Link1">
+  </joint><link name="Link1">
 <inertial>
             <origin xyz="-0.0083034891135278 0.000169963422442479 0.0273090165667047" rpy="0 0 0" />

File: cra_description/urdf/nova2_robot.xacro (robot description, xacro)
@@ -1,6 +1,5 @@
 <?xml version="1.0"?>
 <robot name="nova2_robot" xmlns:xacro="http://www.ros.org/wiki/xacro">
-    <link name="dummy_link" />
-    <link name="base_link">
+  <link name="dummy_link" /><link name="base_link">
     <inertial>
             <origin xyz="1.31739324853774E-05 -7.84959718585273E-06 0.0647773077977383" rpy="0 0 0" />
@@ -24,4 +23,8 @@
         </collision>
     </link>
+  <joint name="dummy_joint" type="fixed">
+      <parent link="dummy_link" />
+      <child  link="base_link" />
+    </joint>
   <link  name="world"/>
   <joint name="world_joint" type="fixed">
@@ -29,14 +32,5 @@
     <parent link="world" />
     <child  link="dummy_link" />
-  </joint>
-  <joint
-    name="dummy_joint"
-    type="fixed">
-    <parent
-      link="dummy_link" />
-    <child
-      link="base_link" />
-  </joint>
-    <link name="Link1">
+  </joint><link name="Link1">
 <inertial>
             <origin xyz="-5.44523391156536E-07 -0.0218722568945782 -0.0236239644661121" rpy="0 0 0" />
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